File: KiCads del proyecto de Electiva (Zorionx_Nivara)/NIVARA_ZorionX.kicad_sch (KiCad schematic)
At the start: 11 parts, among them J6 Screw_Terminal_01x02

Commit message: Esquemas PCB Readys
Parts:
- removed J6, KNY1, KNY13, KNY3, KNY4: Screw_Terminal_01x02, TerminalBlock_Phoenix:TerminalBlock_Phoenix_PT-1,5-2-5.0-H_1x02_P5.00mm_Horizontal, symbol Connector:Screw_Terminal_01x02
- removed KNY12, KNY2: Screw_Terminal_01x04, TerminalBlock_Phoenix:TerminalBlock_Phoenix_PT-1,5-4-5.0-H_1x04_P5.00mm_Horizontal, symbol Connector:Screw_Terminal_01x04
- removed KNY14: Screw_Terminal_01x06, TerminalBlock_Phoenix:TerminalBlock_Phoenix_PT-1,5-6-5.0-H_1x06_P5.00mm_Horizontal, symbol Connector:Screw_Terminal_01x06
- removed KNY5, KNY9: Screw_Terminal_01x03, TerminalBlock_Phoenix:TerminalBlock_Phoenix_PT-1,5-3-3.5-H_1x03_P3.50mm_Horizontal, symbol Connector:Screw_Terminal_01x03
- removed KNYWIFI1: Wifi, symbol Device:Antenna
- added AE1: Antenna, symbol Device:Antenna
- added J1, J2, J4, J7, J8, J9: Screw_Terminal_01x03, symbol Connector:Screw_Terminal_01x03
- added J11, J5: Screw_Terminal_01x02, symbol Connector:Screw_Terminal_01x02
- added J12, J3: Screw_Terminal_01x04, symbol Connector:Screw_Terminal_01x04
- added J6: Screw_Terminal_01x06, symbol Connector:Screw_Terminal_01x06
Connections:
- net GND: now also J11.2 (Pin_2), J12.4 (Pin_4), J3.4 (Pin_4), J4.3 (Pin_3), J5.2 (Pin_2), J7.3 (Pin_3), J9.1 (Pin_1)
- net VCC: now also J11.1 (Pin_1), J8.1 (Pin_1)
- new net NIVARA_BOARD/+10V_AINPUT: J3.1 (Pin_1)
- new net NIVARA_BOARD/+32V_AINPUT: J3.2 (Pin_2)
- new net NIVARA_BOARD/DRY_DINPUT_0: J4.1 (Pin_1)
- new net NIVARA_BOARD/DRY_DINPUT_1: J4.2 (Pin_2)
- new net NIVARA_BOARD/NPN_DINPUT_0: J1.1 (Pin_1)
- new net NIVARA_BOARD/NPN_DINPUT_1: J1.2 (Pin_2)
- new net NIVARA_BOARD/NPN_DOUTPUT_0: J8.2 (Pin_2)
- new net NIVARA_BOARD/NPN_DOUTPUT_1: J8.3 (Pin_3)
- new net NIVARA_BOARD/PNP_DINPUT_0: J2.1 (Pin_1)
- new net NIVARA_BOARD/PNP_DINPUT_1: J2.2 (Pin_2)
- new net NIVARA_BOARD/PNP_DOUTPUT_0: J9.2 (Pin_2)
- new net NIVARA_BOARD/PNP_DOUTPUT_1: J9.3 (Pin_3)
- new net NIVARA_BOARD/RL1_COM: J6.3 (Pin_3)
- new net NIVARA_BOARD/RL1_OUTPUT_NC: J6.2 (Pin_2)
- new net NIVARA_BOARD/RL1_OUTPUT_NO: J6.1 (Pin_1)
- new net NIVARA_BOARD/RL2_COM: J6.6 (Pin_6)
- new net NIVARA_BOARD/RL2_OUTPUT_NC: J6.5 (Pin_5)
- new net NIVARA_BOARD/RL2_OUTPUT_NO: J6.4 (Pin_4)
- new net NIVARA_BOARD/RS485_A: J7.1 (Pin_1)
- new net NIVARA_BOARD/RS485_B: J7.2 (Pin_2)
- new net NIVARA_BOARD/VOLTAGE_AOUTPUT: J12.1 (Pin_1)
- new net NIVARA_BOARD/mA_AINPUT: J3.3 (Pin_3)
- new net NIVARA_BOARD/mA_AOUTPUT+: J12.2 (Pin_2)
- new net NIVARA_BOARD/~{RUN}/STOP: J5.1 (Pin_1)
- new net NPNIN_GND: J1.3 (Pin_3)
- new net PNPIN_GND: J2.3 (Pin_3)
Other:
- removed sheet Board_Nivara
- added sheet NIVARA_BOARD (NIVARA_BOARD.kicad_sch)
- note added: "+24VDC"
- note removed: "24vdc"
- note removed: "Alimentación"
- note removed: "Entrada stop/run (como los PLC)"
- company: Electia_ITLA -> (none)
- title: ZorionX-Nivara -> (none)
