File: KiCads del proyecto de Electiva (Zorionx_Nivara)/Nivara_Zorionx.kicad_pcb (KiCad board)
At the start: 2 copper layers, 107 x 87.7 mm, 20 parts, among them J1 Screw_Terminal_01x02, J12 Screw_Terminal_01x04, J13 Screw_Terminal_01x02, J14 Screw_Terminal_01x06, J2 Screw_Terminal_01x04, J3 Screw_Terminal_01x02, J4 Screw_Terminal_01x02, J5 Screw_Terminal_01x03, J6 Screw_Terminal_01x02, J9 Screw_Terminal_01x03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

Commit message: .
Other:
- copper layers 2 -> 4
Changed lines of the file:
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@@
 	(layers
 		(0 "F.Cu" signal)
+		(4 "In1.Cu" power)
+		(6 "In2.Cu" mixed)
 		(2 "B.Cu" signal)
 		(9 "F.Adhes" user "F.Adhesive")
@@
 	)
 	(setup
+		(stackup
+			(layer "F.SilkS"
+				(type "Top Silk Screen")
+			)
+			(layer "F.Paste"
+				(type "Top Solder Paste")
+			)
+			(layer "F.Mask"
+				(type "Top Solder Mask")
+				(thickness 0.01)
+			)
+			(layer "F.Cu"
+				(type "copper")
+				(thickness 0.035)
+			)
+			(layer "dielectric 1"
+				(type "prepreg")
+				(thickness 0.1)
+				(material "FR4")
+				(epsilon_r 4.5)
+				(loss_tangent 0.02)
+			)
+			(layer "In1.Cu"
+				(type "copper")
+				(thickness 0.035)
+			)
+			(layer "dielectric 2"
+				(type "core")
+				(thickness 1.24)
+				(material "FR4")
+				(epsilon_r 4.5)
+				(loss_tangent 0.02)
+			)
+			(layer "In2.Cu"
+				(type "copper")
+				(thickness 0.035)
+			)
+			(layer "dielectric 3"
+				(type "prepreg")
+				(thickness 0.1)
+				(material "FR4")
+				(epsilon_r 4.5)
+				(loss_tangent 0.02)
+			)
+			(layer "B.Cu"
+				(type "copper")
+				(thickness 0.035)
+			)
+			(layer "B.Mask"
+				(type "Bottom Solder Mask")
+				(thickness 0.01)
+			)
+			(layer "B.Paste"
+				(type "Bottom Solder Paste")
+			)
+			(layer "B.SilkS"
+				(type "Bottom Silk Screen")
+			)
+			(copper_finish "None")
+			(dielectric_constraints no)
+		)
 		(pad_to_mask_clearance 0)
 		(allow_soldermask_bridges_in_footprints no)

Commit message: Esquemas PCB Readys
Parts:
- removed C1: 1uf, Capacitor_SMD:C_0603_1608Metric
- removed R1: R_US, Resistor_SMD:R_0603_1608Metric
- removed the U2 at (158.8, 125.7)
- added D2: SM712_SOT23, Package_TO_SOT_SMD:SOT-23, F.Cu at (199.3, 88.3)
- added D3: SMF24A, Diode_SMD:D_SMF, F.Cu at (196.8, 121.0)
- added D4: 1N4007, Diode_THT:D_DO-41_SOD81_P10.16mm_Horizontal, F.Cu at (166.9, 88.0)
- added D5: SMF24A, Diode_SMD:D_SMF, F.Cu at (168.0, 98.5)
- added D6: SMF24A, Diode_SMD:D_SMF, F.Cu at (183.9, 113.9)
- added D7: SMF24A, Diode_SMD:D_SMF, F.Cu at (183.9, 117.2)
- added JP1: SolderJumper_2_Open, Jumper:SolderJumper-2_P1.3mm_Open_RoundedPad1.0x1.5mm, F.Cu at (208.6, 93.3)
- added K1: G2RL-1, Relay_THT:Relay_SPDT_Omron_G2RL-1, F.Cu at (151.7, 55.0)
- added K2: G2RL-1, Relay_THT:Relay_SPDT_Omron_G2RL-1, F.Cu at (170.1, 54.6)
- added R10: 910, Resistor_SMD:R_0603_1608Metric, F.Cu at (176.9, 116.0)
- added R12: 910, Resistor_SMD:R_0603_1608Metric, F.Cu at (176.9, 118.6)
- added R18: 910, Resistor_SMD:R_0603_1608Metric, F.Cu at (176.9, 103.4)
- added R19: 910, Resistor_SMD:R_0603_1608Metric, F.Cu at (176.9, 105.9)
- added R36: 910, Resistor_SMD:R_0603_1608Metric, F.Cu at (192.8, 89.7)
- added R7: 910, Resistor_SMD:R_0603_1608Metric, F.Cu at (192.8, 87.1)
- added U10: LTV-357TB, Package_SO:SO-4_4.4x3.6mm_P2.54mm, F.Cu at (170.0, 110.2)
- added U11: ~, Riqi_Parts:eSOP-8, F.Cu at (197.8, 113.0)
- added U12: ~, Package_SO:SO-4_4.4x4.3mm_P2.54mm, F.Cu at (185.3, 107.3)
- added U13: ~, Package_SO:SO-4_4.4x4.3mm_P2.54mm, F.Cu at (196.1, 101.4)
- added U14: ~, Package_SO:SO-4_4.4x4.3mm_P2.54mm, F.Cu at (196.1, 107.3)
- added U15: LTV-357TB, Package_SO:SO-4_4.4x3.6mm_P2.54mm, F.Cu at (185.9, 93.9)
- added U2: AP63203WU, Package_TO_SOT_SMD:TSOT-23-6, F.Cu at (209.0, 89.4)
- added U2: AP63203WU, Package_TO_SOT_SMD:TSOT-23-6, F.Cu at (153.9, 99.1)
- added U2: AP63200WU, Package_TO_SOT_SMD:TSOT-23-6, F.Cu at (189.3, 114.6)
- added U3: ~, Riqi_Parts:YLPTEC RSM3485ECHT, F.Cu at (142.4, 123.0)
- added U4: LTV-357TB, Package_SO:SO-4_4.4x3.6mm_P2.54mm, F.Cu at (185.9, 88.6)
- added U4: ~, Riqi_Parts:SOIC127P600X172-14N, F.Cu at (208.8, 103.5)
- added U5: ~, Package_SO:SO-4_4.4x4.3mm_P2.54mm, F.Cu at (185.3, 101.4)
- added U6: ~, Package_SO:SSOP-10-1EP_3.9x4.9mm_P1mm_EP2.1x3.3mm, F.Cu at (169.3, 93.6)
- added U7: LTV-357TB, Package_SO:SO-4_4.4x3.6mm_P2.54mm, F.Cu at (170.0, 117.5)
- added U8: LTV-357TB, Package_SO:SO-4_4.4x3.6mm_P2.54mm, F.Cu at (170.0, 122.8)
- added U9: LTV-357TB, Package_SO:SO-4_4.4x3.6mm_P2.54mm, F.Cu at (170.0, 104.9)
- moved U1 58.4 mm to (117.2, 60.3), turned to -90 degrees
- moved J1 45.1 mm to (53.9, 107.6)
- moved J13 45.1 mm to (41.4, 107.6)
- moved J14 45.1 mm to (93.0, 32.2)
- moved J9 45.1 mm to (54.0, 32.2)
- moved J12 45.1 mm to (67.5, 32.1)
- moved J2 45.1 mm to (65.8, 107.5)
- moved J5 45.1 mm to (41.2, 32.1)
- moved J6 45.1 mm to (105.5, 107.5)
- moved J3 45.1 mm to (118.7, 107.5)
- moved J4 45.1 mm to (90.6, 107.6)
- moved C3 27.1 mm to (147.6, 97.3)
- moved L1 27.1 mm to (148.7, 91.9)
- moved R3 27.1 mm to (161.2, 93.7)
- moved C2 27.1 mm to (154.9, 89.6)
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Connections:
- U1 pad 12: unconnected-(U1-GPIO8/TOUCH8/ADC1_CH7/SUBSPICS1-Pad12) -> /NIVARA_BOARD/PNP_IN_Mod/NPN_Output0
- U1 pad 15: unconnected-(U1-GPIO3/TOUCH3/ADC1_CH2-Pad15) -> /NIVARA_BOARD/RELAY_INTERFACE/RL2_EN
- U1 pad 16: unconnected-(U1-GPIO46-Pad16) -> /NIVARA_BOARD/~{TRANSMIT}/RECEIVE
- U1 pad 17: unconnected-(U1-GPIO9/TOUCH9/ADC1_CH8/FSPIHD/SUBSPIHD-Pad17) -> /NIVARA_BOARD/PNP_IN_Mod/NPN_Output1
- U1 pad 18: unconnected-(U1-GPIO10/TOUCH10/ADC1_CH9/FSPICS0/FSPIIO4/SUBSPICS0-Pad18) -> /NIVARA_BOARD/DRY_INPUT_INTERFACE/DRY_OUT0
- U1 pad 23: unconnected-(U1-GPIO21-Pad23) -> /NIVARA_BOARD/DRY_INPUT_INTERFACE/DRY_OUT1
- U1 pad 24: unconnected-(U1-GPIO47/SPICLK_P/SUBSPICLK_P_DIFF-Pad24) -> /NIVARA_BOARD/RS485_INTERFACE/UART_TX
- U1 pad 25: unconnected-(U1-GPIO48/SPICLK_N/SUBSPICLK_N_DIFF-Pad25) -> /NIVARA_BOARD/RS485_INTERFACE/UART_RX
- U1 pad 26: unconnected-(U1-GPIO45-Pad26) -> /NIVARA_BOARD/NPN_OUT_INTERFACE/NPN_EN1
- U1 pad 28: unconnected-(U1-SPIIO6/GPIO35/FSPID/SUBSPID-Pad28) -> /NIVARA_BOARD/VOLTAGE_AOUT_INTERFACE/SEL
- U1 pad 29: unconnected-(U1-SPIIO7/GPIO36/FSPICLK/SUBSPICLK-Pad29) -> /NIVARA_BOARD/~{RUN}/STOP
- U1 pad 31: unconnected-(U1-GPIO38/FSPIWP/SUBSPIWP-Pad31) -> /NIVARA_BOARD/NPN_OUT_INTERFACE/NPN_EN0
- U1 pad 36: /Board_ZorionX/Driver_RS485/UART_OUT -> unconnected-(U1-U0RXD/GPIO44/CLK_OUT2-Pad36)
- U1 pad 37: /Board_ZorionX/Driver_RS485/UART_R_IN -> unconnected-(U1-U0TXD/GPIO43/CLK_OUT1-Pad37)
- U1 pad 38: unconnected-(U1-GPIO2/TOUCH2/ADC1_CH1-Pad38) -> /NIVARA_BOARD/RELAY_INTERFACE/RL1_EN
- U1 pad 39: unconnected-(U1-GPIO1/TOUCH1/ADC1_CH0-Pad39) -> /NIVARA_BOARD/mA_AINPUT
- U1 pad 4: unconnected-(U1-GPIO4/TOUCH4/ADC1_CH3-Pad4) -> /NIVARA_BOARD/32V_AIN_INTERFACE/32V_ADC
- U1 pad 5: unconnected-(U1-GPIO5/TOUCH5/ADC1_CH4-Pad5) -> /NIVARA_BOARD/10V_AIN_INTERFACE/10V_ADC
- U1 pad 6: unconnected-(U1-GPIO6/TOUCH6/ADC1_CH5-Pad6) -> /NIVARA_BOARD/PNP_OUT_INTERFACE/PNP_EN0
- U1 pad 7: unconnected-(U1-GPIO7/TOUCH7/ADC1_CH6-Pad7) -> /NIVARA_BOARD/PNP_OUT_INTERFACE/PNP_EN1
- U1 pad 8: unconnected-(U1-GPIO15/U0RTS/ADC2_CH4/XTAL_32K_P-Pad8) -> /NIVARA_BOARD/VOLTAGE_AOUT_INTERFACE/SDA
- U1 pad 9: unconnected-(U1-GPIO16/U0CTS/ADC2_CH5/XTAL_32K_N-Pad9) -> /NIVARA_BOARD/VOLTAGE_AOUT_INTERFACE/SCLK
Other:
- board size 107 x 87.7 mm -> 109.1 x 87.7 mm
- copper layers 4 -> 2
