File: KiCads del proyecto de Electiva (Nivara_Zorionx)/Entrada_10v.kicad_sch (KiCad schematic)
At the start: 3 parts

Commit message: Papadio Dame Fuerza 😭
Parts:
- C10: footprint (none) -> Capacitor_SMD:C_0805_2012Metric
- R23: renamed from R16; footprint (none) -> Resistor_SMD:R_0603_1608Metric
- R24: renamed from R17; footprint (none) -> Resistor_SMD:R_0603_1608Metric
Changed lines of the file:
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@@
 		(dnp no)
 		(fields_autoplaced yes)
-		(property "Reference" "R17"
+		(property "Reference" "R24"
 			(at 146.05 80.0099 0)
 			(effects
@@
 			)
 		)
-		(property "Footprint" ""
+		(property "Footprint" "Resistor_SMD:R_0603_1608Metric"
 			(at 141.732 81.28 90)
 			(effects
@@
 			(project "NIVARA"
 				(path "/8290cc18-06d0-4e02-a781-29a61ebc321a/9e4d7a0c-a5eb-4e88-9036-0c35e68b279a/8c13851c-1f51-45db-a0c3-d4fd67e1b6ee"
-					(reference "R17")
-					(unit 1)
-				)
-			)
-			(project "NIVARA_ZorionX_BOARD"
-				(path "/8e19332e-3534-4a04-99a8-04957ac8928f/8c13851c-1f51-45db-a0c3-d4fd67e1b6ee"
-					(reference "R17")
+					(reference "R24")
+					(unit 1)
+				)
+			)
+			(project "NIVARA_ZorionX_BOARD"
+				(path "/8e19332e-3534-4a04-99a8-04957ac8928f/8c13851c-1f51-45db-a0c3-d4fd67e1b6ee"
+					(reference "R?")
 					(unit 1)
 				)
@@
 			)
 		)
-		(property "Footprint" ""
+		(property "Footprint" "Capacitor_SMD:C_0805_2012Metric"
 			(at 153.3652 85.09 0)
 			(effects
@@
 			(project "NIVARA_ZorionX_BOARD"
 				(path "/8e19332e-3534-4a04-99a8-04957ac8928f/8c13851c-1f51-45db-a0c3-d4fd67e1b6ee"
-					(reference "C10")
+					(reference "C?")
 					(unit 1)
 				)
@@
 		(dnp no)
 		(fields_autoplaced yes)
-		(property "Reference" "#PWR041"
+		(property "Reference" "#PWR050"
 			(at 143.51 93.98 0)
 			(effects
@@
 			(project "NIVARA"
 				(path "/8290cc18-06d0-4e02-a781-29a61ebc321a/9e4d7a0c-a5eb-4e88-9036-0c35e68b279a/8c13851c-1f51-45db-a0c3-d4fd67e1b6ee"
-					(reference "#PWR041")
-					(unit 1)
-				)
-			)
-			(project "NIVARA_ZorionX_BOARD"
-				(path "/8e19332e-3534-4a04-99a8-04957ac8928f/8c13851c-1f51-45db-a0c3-d4fd67e1b6ee"
-					(reference "#PWR041")
+					(reference "#PWR050")
+					(unit 1)
+				)
+			)
+			(project "NIVARA_ZorionX_BOARD"
+				(path "/8e19332e-3534-4a04-99a8-04957ac8928f/8c13851c-1f51-45db-a0c3-d4fd67e1b6ee"
+					(reference "#PWR?")
 					(unit 1)
 				)
@@
 		(dnp no)
 		(fields_autoplaced yes)
-		(property "Reference" "R16"
+		(property "Reference" "R23"
 			(at 146.05 68.5799 0)
 			(effects
@@
 			)
 		)
-		(property "Footprint" ""
+		(property "Footprint" "Resistor_SMD:R_0603_1608Metric"
 			(at 141.732 69.85 90)
 			(effects
@@
 			(project "NIVARA"
 				(path "/8290cc18-06d0-4e02-a781-29a61ebc321a/9e4d7a0c-a5eb-4e88-9036-0c35e68b279a/8c13851c-1f51-45db-a0c3-d4fd67e1b6ee"
-					(reference "R16")
-					(unit 1)
-				)
-			)
-			(project "NIVARA_ZorionX_BOARD"
-				(path "/8e19332e-3534-4a04-99a8-04957ac8928f/8c13851c-1f51-45db-a0c3-d4fd67e1b6ee"
-					(reference "R16")
-					(unit 1)
-				)
+					(reference "R23")
+					(unit 1)
+				)
+			)
+			(project "NIVARA_ZorionX_BOARD"
+				(path "/8e19332e-3534-4a04-99a8-04957ac8928f/8c13851c-1f51-45db-a0c3-d4fd67e1b6ee"
+					(reference "R?")
+					(unit 1)
+				)
