File: KiCads del proyecto de Electiva (Nivara_Zorionx)/Entrada_32v.kicad_sch (KiCad schematic)
At the start: 3 parts

Commit message: Papadio Dame Fuerza 😭
Parts:
- C9: footprint (none) -> Capacitor_SMD:C_0805_2012Metric
- R21: renamed from R14; footprint (none) -> Resistor_SMD:R_0603_1608Metric
- R22: renamed from R15; footprint (none) -> Resistor_SMD:R_0603_1608Metric
Changed lines of the file:
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@@
 		(dnp no)
 		(fields_autoplaced yes)
-		(property "Reference" "R15"
+		(property "Reference" "R22"
 			(at 153.67 80.0099 0)
 			(effects
@@
 			)
 		)
-		(property "Footprint" ""
+		(property "Footprint" "Resistor_SMD:R_0603_1608Metric"
 			(at 149.352 81.28 90)
 			(effects
@@
 			(project ""
 				(path "/8290cc18-06d0-4e02-a781-29a61ebc321a/9e4d7a0c-a5eb-4e88-9036-0c35e68b279a/addf1e1e-f652-4279-8cba-01ccd2e4a395"
-					(reference "R15")
-					(unit 1)
-				)
-			)
-			(project "NIVARA_ZorionX_BOARD"
-				(path "/8e19332e-3534-4a04-99a8-04957ac8928f/addf1e1e-f652-4279-8cba-01ccd2e4a395"
-					(reference "R15")
+					(reference "R22")
+					(unit 1)
+				)
+			)
+			(project "NIVARA_ZorionX_BOARD"
+				(path "/8e19332e-3534-4a04-99a8-04957ac8928f/addf1e1e-f652-4279-8cba-01ccd2e4a395"
+					(reference "R?")
 					(unit 1)
 				)
@@
 			)
 		)
-		(property "Footprint" ""
+		(property "Footprint" "Capacitor_SMD:C_0805_2012Metric"
 			(at 162.2552 85.09 0)
 			(effects
@@
 			(project "NIVARA_ZorionX_BOARD"
 				(path "/8e19332e-3534-4a04-99a8-04957ac8928f/addf1e1e-f652-4279-8cba-01ccd2e4a395"
-					(reference "C9")
+					(reference "C?")
 					(unit 1)
 				)
@@
 		(dnp no)
 		(fields_autoplaced yes)
-		(property "Reference" "#PWR038"
+		(property "Reference" "#PWR049"
 			(at 151.13 93.98 0)
 			(effects
@@
 			(project ""
 				(path "/8290cc18-06d0-4e02-a781-29a61ebc321a/9e4d7a0c-a5eb-4e88-9036-0c35e68b279a/addf1e1e-f652-4279-8cba-01ccd2e4a395"
-					(reference "#PWR038")
-					(unit 1)
-				)
-			)
-			(project "NIVARA_ZorionX_BOARD"
-				(path "/8e19332e-3534-4a04-99a8-04957ac8928f/addf1e1e-f652-4279-8cba-01ccd2e4a395"
-					(reference "#PWR038")
+					(reference "#PWR049")
+					(unit 1)
+				)
+			)
+			(project "NIVARA_ZorionX_BOARD"
+				(path "/8e19332e-3534-4a04-99a8-04957ac8928f/addf1e1e-f652-4279-8cba-01ccd2e4a395"
+					(reference "#PWR?")
 					(unit 1)
 				)
@@
 		(dnp no)
 		(fields_autoplaced yes)
-		(property "Reference" "R14"
+		(property "Reference" "R21"
 			(at 153.67 68.5799 0)
 			(effects
@@
 			)
 		)
-		(property "Footprint" ""
+		(property "Footprint" "Resistor_SMD:R_0603_1608Metric"
 			(at 149.352 69.85 90)
 			(effects
@@
 			(project ""
 				(path "/8290cc18-06d0-4e02-a781-29a61ebc321a/9e4d7a0c-a5eb-4e88-9036-0c35e68b279a/addf1e1e-f652-4279-8cba-01ccd2e4a395"
-					(reference "R14")
-					(unit 1)
-				)
-			)
-			(project "NIVARA_ZorionX_BOARD"
-				(path "/8e19332e-3534-4a04-99a8-04957ac8928f/addf1e1e-f652-4279-8cba-01ccd2e4a395"
-					(reference "R14")
-					(unit 1)
-				)
+					(reference "R21")
+					(unit 1)
+				)
+			)
+			(project "NIVARA_ZorionX_BOARD"
+				(path "/8e19332e-3534-4a04-99a8-04957ac8928f/addf1e1e-f652-4279-8cba-01ccd2e4a395"
+					(reference "R?")
+					(unit 1)
+				)
