File: KiCads del proyecto de Electiva (Nivara_Zorionx)/Entrada_dry.kicad_sch (KiCad schematic)
At the start: 6 parts, among them U7 LTV-357TB, U8 LTV-357TB

Commit message: Papadio Dame Fuerza 😭
Parts:
- R19: renamed from R11; footprint (none) -> Resistor_SMD:R_0603_1608Metric
- R20: renamed from R13; footprint (none) -> Resistor_SMD:R_0603_1608Metric
- renumbered R10 to R17, R12 to R18, U7 to U8, U8 to U9
Changed lines of the file:
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@@
 		(dnp no)
 		(fields_autoplaced yes)
-		(property "Reference" "R11"
+		(property "Reference" "R19"
 			(at 163.83 67.3099 0)
 			(effects
@@
 			)
 		)
-		(property "Footprint" ""
+		(property "Footprint" "Resistor_SMD:R_0603_1608Metric"
 			(at 163.068 68.58 90)
 			(effects
@@
 			(project "NIVARA"
 				(path "/8290cc18-06d0-4e02-a781-29a61ebc321a/9e4d7a0c-a5eb-4e88-9036-0c35e68b279a/2ac137b5-1347-46a5-b780-a606790c1a93"
-					(reference "R11")
-					(unit 1)
-				)
-			)
-			(project "NIVARA_ZorionX_BOARD"
-				(path "/8e19332e-3534-4a04-99a8-04957ac8928f/2ac137b5-1347-46a5-b780-a606790c1a93"
-					(reference "R11")
+					(reference "R19")
+					(unit 1)
+				)
+			)
+			(project "NIVARA_ZorionX_BOARD"
+				(path "/8e19332e-3534-4a04-99a8-04957ac8928f/2ac137b5-1347-46a5-b780-a606790c1a93"
+					(reference "R?")
 					(unit 1)
 				)
@@
 		(dnp no)
 		(fields_autoplaced yes)
-		(property "Reference" "#PWR035"
+		(property "Reference" "#PWR046"
 			(at 161.29 66.04 0)
 			(effects
@@
 			(project "NIVARA"
 				(path "/8290cc18-06d0-4e02-a781-29a61ebc321a/9e4d7a0c-a5eb-4e88-9036-0c35e68b279a/2ac137b5-1347-46a5-b780-a606790c1a93"
-					(reference "#PWR035")
-					(unit 1)
-				)
-			)
-			(project "NIVARA_ZorionX_BOARD"
-				(path "/8e19332e-3534-4a04-99a8-04957ac8928f/2ac137b5-1347-46a5-b780-a606790c1a93"
-					(reference "#PWR035")
+					(reference "#PWR046")
+					(unit 1)
+				)
+			)
+			(project "NIVARA_ZorionX_BOARD"
+				(path "/8e19332e-3534-4a04-99a8-04957ac8928f/2ac137b5-1347-46a5-b780-a606790c1a93"
+					(reference "#PWR?")
 					(unit 1)
 				)
@@
 		(dnp no)
 		(fields_autoplaced yes)
-		(property "Reference" "#PWR040"
+		(property "Reference" "#PWR048"
 			(at 165.1 91.44 0)
 			(effects
@@
 			(project "NIVARA"
 				(path "/8290cc18-06d0-4e02-a781-29a61ebc321a/9e4d7a0c-a5eb-4e88-9036-0c35e68b279a/2ac137b5-1347-46a5-b780-a606790c1a93"
-					(reference "#PWR040")
-					(unit 1)
-				)
-			)
-			(project "NIVARA_ZorionX_BOARD"
-				(path "/8e19332e-3534-4a04-99a8-04957ac8928f/2ac137b5-1347-46a5-b780-a606790c1a93"
-					(reference "#PWR040")
+					(reference "#PWR048")
+					(unit 1)
+				)
+			)
+			(project "NIVARA_ZorionX_BOARD"
+				(path "/8e19332e-3534-4a04-99a8-04957ac8928f/2ac137b5-1347-46a5-b780-a606790c1a93"
+					(reference "#PWR?")
 					(unit 1)
 				)
@@
 		(dnp no)
 		(fields_autoplaced yes)
-		(property "Reference" "#PWR036"
+		(property "Reference" "#PWR043"
 			(at 127 76.2 0)
 			(effects
@@
 			(project ""
 				(path "/8290cc18-06d0-4e02-a781-29a61ebc321a/9e4d7a0c-a5eb-4e88-9036-0c35e68b279a/2ac137b5-1347-46a5-b780-a606790c1a93"
-					(reference "#PWR036")
-					(unit 1)
-				)
-			)
-			(project "NIVARA_ZorionX_BOARD"
-				(path "/8e19332e-3534-4a04-99a8-04957ac8928f/2ac137b5-1347-46a5-b780-a606790c1a93"
-					(reference "#PWR036")
+					(reference "#PWR043")
+					(unit 1)
+				)
+			)
+			(project "NIVARA_ZorionX_BOARD"
+				(path "/8e19332e-3534-4a04-99a8-04957ac8928f/2ac137b5-1347-46a5-b780-a606790c1a93"
+					(reference "#PWR?")
 					(unit 1)
 				)
@@
 		(dnp no)
 		(fields_autoplaced yes)
-		(property "Reference" "U7"
+		(property "Reference" "U8"
 			(at 151.13 68.58 0)
 			(effects
@@
 			(project "NIVARA"
 				(path "/8290cc18-06d0-4e02-a781-29a61ebc321a/9e4d7a0c-a5eb-4e88-9036-0c35e68b279a/2ac137b5-1347-46a5-b780-a606790c1a93"
-					(reference "U7")
-					(unit 1)
-				)
-			)
-			(project "NIVARA_ZorionX_BOARD"
-				(path "/8e19332e-3534-4a04-99a8-04957ac8928f/2ac137b5-1347-46a5-b780-a606790c1a93"
-					(reference "U7")
+					(reference "U8")
+					(unit 1)
+				)
+			)
+			(project "NIVARA_ZorionX_BOARD"
+				(path "/8e19332e-3534-4a04-99a8-04957ac8928f/2ac137b5-1347-46a5-b780-a606790c1a93"
+					(reference "U?")
 					(unit 1)
 				)
@@
 		(dnp no)
 		(fields_autoplaced yes)
-		(property "Reference" "R13"
+		(property "Reference" "R20"
 			(at 167.64 92.7099 0)
 			(effects
@@
 			)
 		)
-		(property "Footprint" ""
+		(property "Footprint" "Resistor_SMD:R_0603_1608Metric"
 			(at 166.878 93.98 90)
 			(effects
@@
 			(project "NIVARA"
 				(path "/8290cc18-06d0-4e02-a781-29a61ebc321a/9e4d7a0c-a5eb-4e88-9036-0c35e68b279a/2ac137b5-1347-46a5-b780-a606790c1a93"
-					(reference "R13")
-					(unit 1)
-				)
-			)
-			(project "NIVARA_ZorionX_BOARD"
-				(path "/8e19332e-3534-4a04-99a8-04957ac8928f/2ac137b5-1347-46a5-b780-a606790c1a93"
-					(reference "R13")
+					(reference "R20")
+					(unit 1)
+				)
+			)
+			(project "NIVARA_ZorionX_BOARD"
+				(path "/8e19332e-3534-4a04-99a8-04957ac8928f/2ac137b5-1347-46a5-b780-a606790c1a93"
+					(reference "R?")
 					(unit 1)
 				)
@@
 		(dnp no)
 		(fields_autoplaced yes)
-		(property "Reference" "R10"
+		(property "Reference" "R17"
 			(at 137.16 68.58 90)
 			(effects
@@
 			(project "NIVARA"
 				(path "/8290cc18-06d0-4e02-a781-29a61ebc321a/9e4d7a0c-a5eb-4e88-9036-0c35e68b279a/2ac137b5-1347-46a5-b780-a606790c1a93"
-					(reference "R10")
-					(unit 1)
-				)
-			)
-			(project "NIVARA_ZorionX_BOARD"
-				(path "/8e19332e-3534-4a04-99a8-04957ac8928f/2ac137b5-1347-46a5-b780-a606790c1a93"
-					(reference "R10")
+					(reference "R17")
+					(unit 1)
+				)
+			)
+			(project "NIVARA_ZorionX_BOARD"
+				(path "/8e19332e-3534-4a04-99a8-04957ac8928f/2ac137b5-1347-46a5-b780-a606790c1a93"
+					(reference "R?")
 					(unit 1)
 				)
@@
 		(dnp no)
 		(fields_autoplaced yes)
-		(property "Reference" "R12"
+		(property "Reference" "R18"
 			(at 140.97 93.98 90)
 			(effects
@@
 			(project "NIVARA"
 				(path "/8290cc18-06d0-4e02-a781-29a61ebc321a/9e4d7a0c-a5eb-4e88-9036-0c35e68b279a/2ac137b5-1347-46a5-b780-a606790c1a93"
-					(reference "R12")
-					(unit 1)
-				)
-			)
-			(project "NIVARA_ZorionX_BOARD"
-				(path "/8e19332e-3534-4a04-99a8-04957ac8928f/2ac137b5-1347-46a5-b780-a606790c1a93"
-					(reference "R12")
+					(reference "R18")
+					(unit 1)
+				)
+			)
+			(project "NIVARA_ZorionX_BOARD"
+				(path "/8e19332e-3534-4a04-99a8-04957ac8928f/2ac137b5-1347-46a5-b780-a606790c1a93"
+					(reference "R?")
 					(unit 1)
 				)
@@
 		(dnp no)
 		(fields_autoplaced yes)
-		(property "Reference" "#PWR034"
+		(property "Reference" "#PWR045"
 			(at 160.02 90.17 0)
 			(effects
@@
 			(project "NIVARA"
 				(path "/8290cc18-06d0-4e02-a781-29a61ebc321a/9e4d7a0c-a5eb-4e88-9036-0c35e68b279a/2ac137b5-1347-46a5-b780-a606790c1a93"
-					(reference "#PWR034")
-					(unit 1)
-				)
-			)
-			(project "NIVARA_ZorionX_BOARD"
-				(path "/8e19332e-3534-4a04-99a8-04957ac8928f/2ac137b5-1347-46a5-b780-a606790c1a93"
-					(reference "#PWR034")
+					(reference "#PWR045")
+					(unit 1)
+				)
+			)
+			(project "NIVARA_ZorionX_BOARD"
+				(path "/8e19332e-3534-4a04-99a8-04957ac8928f/2ac137b5-1347-46a5-b780-a606790c1a93"
+					(reference "#PWR?")
 					(unit 1)
 				)
@@
 		(dnp no)
 		(fields_autoplaced yes)
-		(property "Reference" "#PWR039"
+		(property "Reference" "#PWR047"
 			(at 163.83 115.57 0)
 			(effects
@@
 			(project "NIVARA"
 				(path "/8290cc18-06d0-4e02-a781-29a61ebc321a/9e4d7a0c-a5eb-4e88-9036-0c35e68b279a/2ac137b5-1347-46a5-b780-a606790c1a93"
-					(reference "#PWR039")
-					(unit 1)
-				)
-			)
-			(project "NIVARA_ZorionX_BOARD"
-				(path "/8e19332e-3534-4a04-99a8-04957ac8928f/2ac137b5-1347-46a5-b780-a606790c1a93"
-					(reference "#PWR039")
+					(reference "#PWR047")
+					(unit 1)
+				)
+			)
+			(project "NIVARA_ZorionX_BOARD"
+				(path "/8e19332e-3534-4a04-99a8-04957ac8928f/2ac137b5-1347-46a5-b780-a606790c1a93"
+					(reference "#PWR?")
 					(unit 1)
 				)
@@
 		(dnp no)
 		(fields_autoplaced yes)
-		(property "Reference" "U8"
+		(property "Reference" "U9"
 			(at 154.94 93.98 0)
 			(effects
@@
 			(project "NIVARA"
 				(path "/8290cc18-06d0-4e02-a781-29a61ebc321a/9e4d7a0c-a5eb-4e88-9036-0c35e68b279a/2ac137b5-1347-46a5-b780-a606790c1a93"
-					(reference "U8")
-					(unit 1)
-				)
-			)
-			(project "NIVARA_ZorionX_BOARD"
-				(path "/8e19332e-3534-4a04-99a8-04957ac8928f/2ac137b5-1347-46a5-b780-a606790c1a93"
-					(reference "U8")
+					(reference "U9")
+					(unit 1)
+				)
+			)
+			(project "NIVARA_ZorionX_BOARD"
+				(path "/8e19332e-3534-4a04-99a8-04957ac8928f/2ac137b5-1347-46a5-b780-a606790c1a93"
+					(reference "U?")
 					(unit 1)
 				)
@@
 		(dnp no)
 		(fields_autoplaced yes)
-		(property "Reference" "#PWR037"
+		(property "Reference" "#PWR044"
 			(at 130.81 101.6 0)
 			(effects
@@
 			(project "NIVARA"
 				(path "/8290cc18-06d0-4e02-a781-29a61ebc321a/9e4d7a0c-a5eb-4e88-9036-0c35e68b279a/2ac137b5-1347-46a5-b780-a606790c1a93"
-					(reference "#PWR037")
-					(unit 1)
-				)
-			)
-			(project "NIVARA_ZorionX_BOARD"
-				(path "/8e19332e-3534-4a04-99a8-04957ac8928f/2ac137b5-1347-46a5-b780-a606790c1a93"
-					(reference "#PWR037")
-					(unit 1)
-				)
+					(reference "#PWR044")
+					(unit 1)
+				)
+			)
+			(project "NIVARA_ZorionX_BOARD"
+				(path "/8e19332e-3534-4a04-99a8-04957ac8928f/2ac137b5-1347-46a5-b780-a606790c1a93"
+					(reference "#PWR?")
+					(unit 1)
+				)
