File: KiCads del proyecto de Electiva (Nivara_Zorionx)/Entradas_NPN.kicad_sch (KiCad schematic)
At the start: 6 parts, among them U10 LTV-357TB, U9 LTV-357TB

Commit message: Papadio Dame Fuerza 😭
Parts:
- R11: renamed from R20; footprint (none) -> Resistor_SMD:R_0603_1608Metric
- R12: renamed from R21; footprint (none) -> Resistor_SMD:R_0603_1608Metric
- renumbered R19 to R10, R18 to R9, U9 to U4, U10 to U5
