File: KiCads del proyecto de Electiva (Nivara_Zorionx)/Entradas_PNP.kicad_sch (KiCad schematic)
At the start: 6 parts, among them U10 LTV-357TB, U9 LTV-357TB

Commit message: Papadio Dame Fuerza 😭
Parts:
- removed R18, R19: 910, Resistor_SMD:R_0603_1608Metric, symbol Device:R
- removed R20, R21: 412, symbol Device:R
- removed U10, U9: LTV-357TB, Package_SO:SO-4_4.4x3.6mm_P2.54mm, symbol Isolator:LTV-357T
- added R26, R27: 910, Resistor_SMD:R_0603_1608Metric, symbol Device:R
- added R28, R29: 412, Resistor_SMD:R_0603_1608Metric, symbol Device:R
- added U11, U12: LTV-357TB, Package_SO:SO-4_4.4x3.6mm_P2.54mm, symbol Isolator:LTV-357T
Connections:
- net +3.3V: now also R28.2, R29.2
- net GND: now also U11.3, U12.3
- net NPN_Input0: now also R26.1
- net NPN_Input1: now also R27.1
- net NPN_Output0: now also R28.1, U11.4
- net NPN_Output1: now also R29.1, U12.4
- net PNPIN_GND: now also U11.2, U12.2
- new net: R27.2, U12.1
- new net: R26.2, U11.1
