File: KiCads del proyecto de Electiva (Nivara_Zorionx)/Modulo de alimentación de diferencia de potencial.kicad_sch (KiCad schematic)
At the start: 12 parts, among them U2 AP63200WU

Commit message: Papadio Dame Fuerza 😭
Parts:
- C2: renamed from C3; footprint (none) -> Capacitor_SMD:C_0805_2012Metric
- C3: renamed from C2; footprint (none) -> Capacitor_SMD:C_0805_2012Metric
- C4: renamed from C6; footprint (none) -> Capacitor_SMD:C_0805_2012Metric
- C5: renamed from C4; footprint (none) -> Capacitor_SMD:C_0805_2012Metric
- C6: renamed from C5; footprint (none) -> Capacitor_SMD:C_0805_2012Metric
- L1: footprint (none) -> Inductor_SMD:L_1206_3216Metric
- R5: renamed from R2; footprint (none) -> Resistor_SMD:R_0603_1608Metric
- R6: renamed from R3; footprint (none) -> Resistor_SMD:R_0603_1608Metric
- renumbered D7 to D1, D6 to D2
