File: KiCads del proyecto de Electiva (Nivara_Zorionx)/Modulo_RS485.kicad_sch (KiCad schematic)
At the start: 4 parts

Commit message: Papadio Dame Fuerza 😭
Parts:
- R7: renamed from R24; footprint (none) -> Resistor_SMD:R_0603_1608Metric
- R8: renamed from R25; footprint (none) -> Resistor_SMD:R_0603_1608Metric
- renumbered D2 to D3
Changed lines of the file:
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@@
 		(dnp no)
 		(fields_autoplaced yes)
-		(property "Reference" "#PWR16"
+		(property "Reference" "#PWR024"
 			(at 116.84 95.25 0)
 			(effects
@@
 			(project ""
 				(path "/8290cc18-06d0-4e02-a781-29a61ebc321a/9e4d7a0c-a5eb-4e88-9036-0c35e68b279a/43a112db-786f-42fb-8db3-67286b51ed8f"
-					(reference "#PWR16")
-					(unit 1)
-				)
-			)
-			(project "NIVARA_ZorionX_BOARD"
-				(path "/8e19332e-3534-4a04-99a8-04957ac8928f/43a112db-786f-42fb-8db3-67286b51ed8f"
-					(reference "#PWR16")
+					(reference "#PWR024")
+					(unit 1)
+				)
+			)
+			(project "NIVARA_ZorionX_BOARD"
+				(path "/8e19332e-3534-4a04-99a8-04957ac8928f/43a112db-786f-42fb-8db3-67286b51ed8f"
+					(reference "#PWR?")
 					(unit 1)
 				)
@@
 		(dnp no)
 		(fields_autoplaced yes)
-		(property "Reference" "R24"
+		(property "Reference" "R7"
 			(at 142.24 64.77 90)
 			(effects
@@
 			)
 		)
-		(property "Footprint" ""
+		(property "Footprint" "Resistor_SMD:R_0603_1608Metric"
 			(at 142.24 72.898 90)
 			(effects
@@
 			(project ""
 				(path "/8290cc18-06d0-4e02-a781-29a61ebc321a/9e4d7a0c-a5eb-4e88-9036-0c35e68b279a/43a112db-786f-42fb-8db3-67286b51ed8f"
-					(reference "R24")
-					(unit 1)
-				)
-			)
-			(project "NIVARA_ZorionX_BOARD"
-				(path "/8e19332e-3534-4a04-99a8-04957ac8928f/43a112db-786f-42fb-8db3-67286b51ed8f"
-					(reference "R24")
+					(reference "R7")
+					(unit 1)
+				)
+			)
+			(project "NIVARA_ZorionX_BOARD"
+				(path "/8e19332e-3534-4a04-99a8-04957ac8928f/43a112db-786f-42fb-8db3-67286b51ed8f"
+					(reference "R?")
 					(unit 1)
 				)
@@
 			(project "NIVARA_ZorionX_BOARD"
 				(path "/8e19332e-3534-4a04-99a8-04957ac8928f/43a112db-786f-42fb-8db3-67286b51ed8f"
-					(reference "U3")
+					(reference "U?")
 					(unit 1)
 				)
@@
 		(dnp no)
 		(fields_autoplaced yes)
-		(property "Reference" "D2"
+		(property "Reference" "D3"
 			(at 158.75 78.74 0)
 			(effects
@@
 			(project ""
 				(path "/8290cc18-06d0-4e02-a781-29a61ebc321a/9e4d7a0c-a5eb-4e88-9036-0c35e68b279a/43a112db-786f-42fb-8db3-67286b51ed8f"
-					(reference "D2")
-					(unit 1)
-				)
-			)
-			(project "NIVARA_ZorionX_BOARD"
-				(path "/8e19332e-3534-4a04-99a8-04957ac8928f/43a112db-786f-42fb-8db3-67286b51ed8f"
-					(reference "D2")
+					(reference "D3")
+					(unit 1)
+				)
+			)
+			(project "NIVARA_ZorionX_BOARD"
+				(path "/8e19332e-3534-4a04-99a8-04957ac8928f/43a112db-786f-42fb-8db3-67286b51ed8f"
+					(reference "D?")
 					(unit 1)
 				)
@@
 		(on_board yes)
 		(dnp no)
-		(property "Reference" "R25"
+		(property "Reference" "R8"
 			(at 142.24 81.28 90)
 			(effects
@@
 			)
 		)
-		(property "Footprint" ""
+		(property "Footprint" "Resistor_SMD:R_0603_1608Metric"
 			(at 142.24 73.152 90)
 			(effects
@@
 			(project "NIVARA"
 				(path "/8290cc18-06d0-4e02-a781-29a61ebc321a/9e4d7a0c-a5eb-4e88-9036-0c35e68b279a/43a112db-786f-42fb-8db3-67286b51ed8f"
-					(reference "R25")
-					(unit 1)
-				)
-			)
-			(project "NIVARA_ZorionX_BOARD"
-				(path "/8e19332e-3534-4a04-99a8-04957ac8928f/43a112db-786f-42fb-8db3-67286b51ed8f"
-					(reference "R25")
+					(reference "R8")
+					(unit 1)
+				)
+			)
+			(project "NIVARA_ZorionX_BOARD"
+				(path "/8e19332e-3534-4a04-99a8-04957ac8928f/43a112db-786f-42fb-8db3-67286b51ed8f"
+					(reference "R?")
 					(unit 1)
 				)
@@
 		(dnp no)
 		(fields_autoplaced yes)
-		(property "Reference" "#PWR17"
+		(property "Reference" "#PWR025"
 			(at 120.65 59.69 0)
 			(effects
@@
 			(project ""
 				(path "/8290cc18-06d0-4e02-a781-29a61ebc321a/9e4d7a0c-a5eb-4e88-9036-0c35e68b279a/43a112db-786f-42fb-8db3-67286b51ed8f"
-					(reference "#PWR17")
-					(unit 1)
-				)
-			)
-			(project "NIVARA_ZorionX_BOARD"
-				(path "/8e19332e-3534-4a04-99a8-04957ac8928f/43a112db-786f-42fb-8db3-67286b51ed8f"
-					(reference "#PWR17")
+					(reference "#PWR025")
+					(unit 1)
+				)
+			)
+			(project "NIVARA_ZorionX_BOARD"
+				(path "/8e19332e-3534-4a04-99a8-04957ac8928f/43a112db-786f-42fb-8db3-67286b51ed8f"
+					(reference "#PWR?")
 					(unit 1)
 				)
@@
 		(dnp no)
 		(fields_autoplaced yes)
-		(property "Reference" "#PWR052"
+		(property "Reference" "#PWR026"
 			(at 158.75 97.79 0)
 			(effects
@@
 			(project "NIVARA"
 				(path "/8290cc18-06d0-4e02-a781-29a61ebc321a/9e4d7a0c-a5eb-4e88-9036-0c35e68b279a/43a112db-786f-42fb-8db3-67286b51ed8f"
-					(reference "#PWR052")
-					(unit 1)
-				)
-			)
-			(project "NIVARA_ZorionX_BOARD"
-				(path "/8e19332e-3534-4a04-99a8-04957ac8928f/43a112db-786f-42fb-8db3-67286b51ed8f"
-					(reference "#PWR052")
-					(unit 1)
-				)
+					(reference "#PWR026")
+					(unit 1)
+				)
+			)
+			(project "NIVARA_ZorionX_BOARD"
+				(path "/8e19332e-3534-4a04-99a8-04957ac8928f/43a112db-786f-42fb-8db3-67286b51ed8f"
+					(reference "#PWR?")
+					(unit 1)
+				)
