File: KiCads del proyecto de Electiva (Nivara_Zorionx)/Modulo_Relay.kicad_sch (KiCad schematic)
At the start: 3 parts, among them K1 G2RL-1, K2 G2RL-1

Commit message: Papadio Dame Fuerza 😭
Parts:
- renumbered Q2 to Q1
Changed lines of the file:
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@@
 		(dnp no)
 		(fields_autoplaced yes)
-		(property "Reference" "#PWR021"
+		(property "Reference" "#PWR030"
 			(at 125.73 124.46 0)
 			(effects
@@
 			(project "NIVARA"
 				(path "/8290cc18-06d0-4e02-a781-29a61ebc321a/9e4d7a0c-a5eb-4e88-9036-0c35e68b279a/86b88fb6-54fe-4cca-9b3c-121214f029ac"
-					(reference "#PWR021")
-					(unit 1)
-				)
-			)
-			(project "NIVARA_ZorionX_BOARD"
-				(path "/8e19332e-3534-4a04-99a8-04957ac8928f/86b88fb6-54fe-4cca-9b3c-121214f029ac"
-					(reference "#PWR021")
+					(reference "#PWR030")
+					(unit 1)
+				)
+			)
+			(project "NIVARA_ZorionX_BOARD"
+				(path "/8e19332e-3534-4a04-99a8-04957ac8928f/86b88fb6-54fe-4cca-9b3c-121214f029ac"
+					(reference "#PWR?")
 					(unit 1)
 				)
@@
 			(project "NIVARA_ZorionX_BOARD"
 				(path "/8e19332e-3534-4a04-99a8-04957ac8928f/86b88fb6-54fe-4cca-9b3c-121214f029ac"
-					(reference "K1")
+					(reference "K?")
 					(unit 1)
 				)
@@
 		(dnp no)
 		(fields_autoplaced yes)
-		(property "Reference" "#PWR019"
+		(property "Reference" "#PWR027"
 			(at 109.22 107.95 0)
 			(effects
@@
 			(project "NIVARA"
 				(path "/8290cc18-06d0-4e02-a781-29a61ebc321a/9e4d7a0c-a5eb-4e88-9036-0c35e68b279a/86b88fb6-54fe-4cca-9b3c-121214f029ac"
-					(reference "#PWR019")
-					(unit 1)
-				)
-			)
-			(project "NIVARA_ZorionX_BOARD"
-				(path "/8e19332e-3534-4a04-99a8-04957ac8928f/86b88fb6-54fe-4cca-9b3c-121214f029ac"
-					(reference "#PWR019")
+					(reference "#PWR027")
+					(unit 1)
+				)
+			)
+			(project "NIVARA_ZorionX_BOARD"
+				(path "/8e19332e-3534-4a04-99a8-04957ac8928f/86b88fb6-54fe-4cca-9b3c-121214f029ac"
+					(reference "#PWR?")
 					(unit 1)
 				)
@@
 		(exclude_from_sim no)
 		(in_bom yes)
-		(on_board yes)
-		(dnp no)
-		(fields_autoplaced yes)
-		(property "Reference" "Q2"
+		(on_board no)
+		(dnp no)
+		(fields_autoplaced yes)
+		(property "Reference" "Q1"
 			(at 111.3633 104.14 0)
 			(effects
@@
 			(project ""
 				(path "/8290cc18-06d0-4e02-a781-29a61ebc321a/9e4d7a0c-a5eb-4e88-9036-0c35e68b279a/86b88fb6-54fe-4cca-9b3c-121214f029ac"
-					(reference "Q2")
-					(unit 1)
-				)
-			)
-			(project "NIVARA_ZorionX_BOARD"
-				(path "/8e19332e-3534-4a04-99a8-04957ac8928f/86b88fb6-54fe-4cca-9b3c-121214f029ac"
-					(reference "Q2")
+					(reference "Q1")
+					(unit 1)
+				)
+			)
+			(project "NIVARA_ZorionX_BOARD"
+				(path "/8e19332e-3534-4a04-99a8-04957ac8928f/86b88fb6-54fe-4cca-9b3c-121214f029ac"
+					(reference "Q?")
 					(unit 1)
 				)
@@
 		(dnp no)
 		(fields_autoplaced yes)
-		(property "Reference" "#PWR20"
+		(property "Reference" "#PWR029"
 			(at 120.65 91.44 0)
 			(effects
@@
 			(project ""
 				(path "/8290cc18-06d0-4e02-a781-29a61ebc321a/9e4d7a0c-a5eb-4e88-9036-0c35e68b279a/86b88fb6-54fe-4cca-9b3c-121214f029ac"
-					(reference "#PWR20")
-					(unit 1)
-				)
-			)
-			(project "NIVARA_ZorionX_BOARD"
-				(path "/8e19332e-3534-4a04-99a8-04957ac8928f/86b88fb6-54fe-4cca-9b3c-121214f029ac"
-					(reference "#PWR20")
+					(reference "#PWR029")
+					(unit 1)
+				)
+			)
+			(project "NIVARA_ZorionX_BOARD"
+				(path "/8e19332e-3534-4a04-99a8-04957ac8928f/86b88fb6-54fe-4cca-9b3c-121214f029ac"
+					(reference "#PWR?")
 					(unit 1)
 				)
@@
 		(dnp no)
 		(fields_autoplaced yes)
-		(property "Reference" "#PWR18"
+		(property "Reference" "#PWR028"
 			(at 109.22 130.81 0)
 			(effects
@@
 			(project ""
 				(path "/8290cc18-06d0-4e02-a781-29a61ebc321a/9e4d7a0c-a5eb-4e88-9036-0c35e68b279a/86b88fb6-54fe-4cca-9b3c-121214f029ac"
-					(reference "#PWR18")
-					(unit 1)
-				)
-			)
-			(project "NIVARA_ZorionX_BOARD"
-				(path "/8e19332e-3534-4a04-99a8-04957ac8928f/86b88fb6-54fe-4cca-9b3c-121214f029ac"
-					(reference "#PWR18")
+					(reference "#PWR028")
+					(unit 1)
+				)
+			)
+			(project "NIVARA_ZorionX_BOARD"
+				(path "/8e19332e-3534-4a04-99a8-04957ac8928f/86b88fb6-54fe-4cca-9b3c-121214f029ac"
+					(reference "#PWR?")
 					(unit 1)
 				)
@@
 			(project "NIVARA_ZorionX_BOARD"
 				(path "/8e19332e-3534-4a04-99a8-04957ac8928f/86b88fb6-54fe-4cca-9b3c-121214f029ac"
-					(reference "K2")
-					(unit 1)
-				)
+					(reference "K?")
+					(unit 1)
+				)
