File: KiCads del proyecto de Electiva (Nivara_Zorionx)/NIVARA_ZorionX_BOARD.kicad_sch (KiCad schematic)
At the start: 6 parts, among them U1 ESP32-S3-WROOM-1

Commit message: Papadio Dame Fuerza 😭
Parts:
- renumbered C1 to C310, R22 to R300, R1 to R310, R31 to R320, R32 to R330
Changed lines of the file:
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@@
 		(dnp no)
 		(fields_autoplaced yes)
-		(property "Reference" "R?"
+		(property "Reference" "R330"
 			(at 162.56 115.5699 0)
 			(effects
@@
 			(project "NIVARA_ZorionX_BOARD"
 				(path "/8e19332e-3534-4a04-99a8-04957ac8928f"
-					(reference "R?")
+					(reference "R330")
 					(unit 1)
 				)
@@
 		(dnp no)
 		(fields_autoplaced yes)
-		(property "Reference" "R?"
+		(property "Reference" "R310"
 			(at 165.1 73.6599 0)
 			(effects
@@
 			(project "NIVARA_ZorionX_BOARD"
 				(path "/8e19332e-3534-4a04-99a8-04957ac8928f"
-					(reference "R?")
+					(reference "R310")
 					(unit 1)
 				)
@@
 		(on_board yes)
 		(dnp no)
-		(property "Reference" "C?"
+		(property "Reference" "C310"
 			(at 153.67 76.2001 0)
 			(effects
@@
 			(project "NIVARA_ZorionX_BOARD"
 				(path "/8e19332e-3534-4a04-99a8-04957ac8928f"
-					(reference "C?")
+					(reference "C310")
 					(unit 1)
 				)
@@
 		(dnp no)
 		(fields_autoplaced yes)
-		(property "Reference" "R?"
+		(property "Reference" "R320"
 			(at 154.94 115.5699 0)
 			(effects
@@
 			(project "NIVARA_ZorionX_BOARD"
 				(path "/8e19332e-3534-4a04-99a8-04957ac8928f"
-					(reference "R?")
+					(reference "R320")
 					(unit 1)
 				)
@@
 		(dnp no)
 		(fields_autoplaced yes)
-		(property "Reference" "R?"
+		(property "Reference" "R300"
 			(at 147.32 143.5099 0)
 			(effects
@@
 			(project "NIVARA_ZorionX_BOARD"
 				(path "/8e19332e-3534-4a04-99a8-04957ac8928f"
-					(reference "R?")
-					(unit 1)
-				)
+					(reference "R300")
+					(unit 1)
+				)
