File: KiCads del proyecto de Electiva (Nivara_Zorionx)/Salida_NPN.kicad_sch (KiCad schematic)
At the start: 4 parts

Commit message: Papadio Dame Fuerza 😭
Parts:
- R15: renamed from R4; footprint (none) -> Resistor_SMD:R_0603_1608Metric
- R16: renamed from R26; footprint (none) -> Resistor_SMD:R_0603_1608Metric
- renumbered U5 to U6, U12 to U7
Changed lines of the file:
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@@
 		(dnp no)
 		(fields_autoplaced yes)
-		(property "Reference" "R26"
+		(property "Reference" "R16"
 			(at 172.72 81.28 90)
 			(effects
@@
 			)
 		)
-		(property "Footprint" ""
+		(property "Footprint" "Resistor_SMD:R_0603_1608Metric"
 			(at 172.72 89.408 90)
 			(effects
@@
 			(project "NIVARA"
 				(path "/8290cc18-06d0-4e02-a781-29a61ebc321a/9e4d7a0c-a5eb-4e88-9036-0c35e68b279a/70c9f439-c648-496e-a774-7d3c213f4c72"
-					(reference "R26")
-					(unit 1)
-				)
-			)
-			(project "NIVARA_ZorionX_BOARD"
-				(path "/8e19332e-3534-4a04-99a8-04957ac8928f/70c9f439-c648-496e-a774-7d3c213f4c72"
-					(reference "R26")
+					(reference "R16")
+					(unit 1)
+				)
+			)
+			(project "NIVARA_ZorionX_BOARD"
+				(path "/8e19332e-3534-4a04-99a8-04957ac8928f/70c9f439-c648-496e-a774-7d3c213f4c72"
+					(reference "R?")
 					(unit 1)
 				)
@@
 		(dnp no)
 		(fields_autoplaced yes)
-		(property "Reference" "#PWR023"
+		(property "Reference" "#PWR039"
 			(at 180.34 81.28 0)
 			(effects
@@
 			(project "NIVARA"
 				(path "/8290cc18-06d0-4e02-a781-29a61ebc321a/9e4d7a0c-a5eb-4e88-9036-0c35e68b279a/70c9f439-c648-496e-a774-7d3c213f4c72"
-					(reference "#PWR023")
-					(unit 1)
-				)
-			)
-			(project "NIVARA_ZorionX_BOARD"
-				(path "/8e19332e-3534-4a04-99a8-04957ac8928f/70c9f439-c648-496e-a774-7d3c213f4c72"
-					(reference "#PWR023")
+					(reference "#PWR039")
+					(unit 1)
+				)
+			)
+			(project "NIVARA_ZorionX_BOARD"
+				(path "/8e19332e-3534-4a04-99a8-04957ac8928f/70c9f439-c648-496e-a774-7d3c213f4c72"
+					(reference "#PWR?")
 					(unit 1)
 				)
@@
 		(dnp no)
 		(fields_autoplaced yes)
-		(property "Reference" "#PWR024"
+		(property "Reference" "#PWR042"
 			(at 200.66 102.87 0)
 			(effects
@@
 			(project "NIVARA"
 				(path "/8290cc18-06d0-4e02-a781-29a61ebc321a/9e4d7a0c-a5eb-4e88-9036-0c35e68b279a/70c9f439-c648-496e-a774-7d3c213f4c72"
-					(reference "#PWR024")
-					(unit 1)
-				)
-			)
-			(project "NIVARA_ZorionX_BOARD"
-				(path "/8e19332e-3534-4a04-99a8-04957ac8928f/70c9f439-c648-496e-a774-7d3c213f4c72"
-					(reference "#PWR024")
+					(reference "#PWR042")
+					(unit 1)
+				)
+			)
+			(project "NIVARA_ZorionX_BOARD"
+				(path "/8e19332e-3534-4a04-99a8-04957ac8928f/70c9f439-c648-496e-a774-7d3c213f4c72"
+					(reference "#PWR?")
 					(unit 1)
 				)
@@
 		(dnp no)
 		(fields_autoplaced yes)
-		(property "Reference" "#PWR053"
+		(property "Reference" "#PWR041"
 			(at 200.66 81.28 0)
 			(effects
@@
 			(project "NIVARA"
 				(path "/8290cc18-06d0-4e02-a781-29a61ebc321a/9e4d7a0c-a5eb-4e88-9036-0c35e68b279a/70c9f439-c648-496e-a774-7d3c213f4c72"
-					(reference "#PWR053")
-					(unit 1)
-				)
-			)
-			(project "NIVARA_ZorionX_BOARD"
-				(path "/8e19332e-3534-4a04-99a8-04957ac8928f/70c9f439-c648-496e-a774-7d3c213f4c72"
-					(reference "#PWR053")
+					(reference "#PWR041")
+					(unit 1)
+				)
+			)
+			(project "NIVARA_ZorionX_BOARD"
+				(path "/8e19332e-3534-4a04-99a8-04957ac8928f/70c9f439-c648-496e-a774-7d3c213f4c72"
+					(reference "#PWR?")
 					(unit 1)
 				)
@@
 		(dnp no)
 		(fields_autoplaced yes)
-		(property "Reference" "#PWR027"
+		(property "Reference" "#PWR040"
 			(at 180.34 102.87 0)
 			(effects
@@
 			(project "NIVARA"
 				(path "/8290cc18-06d0-4e02-a781-29a61ebc321a/9e4d7a0c-a5eb-4e88-9036-0c35e68b279a/70c9f439-c648-496e-a774-7d3c213f4c72"
-					(reference "#PWR027")
-					(unit 1)
-				)
-			)
-			(project "NIVARA_ZorionX_BOARD"
-				(path "/8e19332e-3534-4a04-99a8-04957ac8928f/70c9f439-c648-496e-a774-7d3c213f4c72"
-					(reference "#PWR027")
+					(reference "#PWR040")
+					(unit 1)
+				)
+			)
+			(project "NIVARA_ZorionX_BOARD"
+				(path "/8e19332e-3534-4a04-99a8-04957ac8928f/70c9f439-c648-496e-a774-7d3c213f4c72"
+					(reference "#PWR?")
 					(unit 1)
 				)
@@
 		(dnp no)
 		(fields_autoplaced yes)
-		(property "Reference" "R4"
+		(property "Reference" "R15"
 			(at 172.72 59.69 90)
 			(effects
@@
 			)
 		)
-		(property "Footprint" ""
+		(property "Footprint" "Resistor_SMD:R_0603_1608Metric"
 			(at 172.72 67.818 90)
 			(effects
@@
 			(project "NIVARA"
 				(path "/8290cc18-06d0-4e02-a781-29a61ebc321a/9e4d7a0c-a5eb-4e88-9036-0c35e68b279a/70c9f439-c648-496e-a774-7d3c213f4c72"
-					(reference "R4")
-					(unit 1)
-				)
-			)
-			(project "NIVARA_ZorionX_BOARD"
-				(path "/8e19332e-3534-4a04-99a8-04957ac8928f/70c9f439-c648-496e-a774-7d3c213f4c72"
-					(reference "R4")
+					(reference "R15")
+					(unit 1)
+				)
+			)
+			(project "NIVARA_ZorionX_BOARD"
+				(path "/8e19332e-3534-4a04-99a8-04957ac8928f/70c9f439-c648-496e-a774-7d3c213f4c72"
+					(reference "R?")
 					(unit 1)
 				)
@@
 		(dnp no)
 		(fields_autoplaced yes)
-		(property "Reference" "U12"
+		(property "Reference" "U7"
 			(at 190.5 82.55 0)
 			(effects
@@
 			(project "NIVARA"
 				(path "/8290cc18-06d0-4e02-a781-29a61ebc321a/9e4d7a0c-a5eb-4e88-9036-0c35e68b279a/70c9f439-c648-496e-a774-7d3c213f4c72"
-					(reference "U12")
-					(unit 1)
-				)
-			)
-			(project "NIVARA_ZorionX_BOARD"
-				(path "/8e19332e-3534-4a04-99a8-04957ac8928f/70c9f439-c648-496e-a774-7d3c213f4c72"
-					(reference "U12")
+					(reference "U7")
+					(unit 1)
+				)
+			)
+			(project "NIVARA_ZorionX_BOARD"
+				(path "/8e19332e-3534-4a04-99a8-04957ac8928f/70c9f439-c648-496e-a774-7d3c213f4c72"
+					(reference "U?")
 					(unit 1)
 				)
@@
 		(dnp no)
 		(fields_autoplaced yes)
-		(property "Reference" "U5"
+		(property "Reference" "U6"
 			(at 190.5 60.96 0)
 			(effects
@@
 			(project "NIVARA"
 				(path "/8290cc18-06d0-4e02-a781-29a61ebc321a/9e4d7a0c-a5eb-4e88-9036-0c35e68b279a/70c9f439-c648-496e-a774-7d3c213f4c72"
-					(reference "U5")
-					(unit 1)
-				)
-			)
-			(project "NIVARA_ZorionX_BOARD"
-				(path "/8e19332e-3534-4a04-99a8-04957ac8928f/70c9f439-c648-496e-a774-7d3c213f4c72"
-					(reference "U5")
-					(unit 1)
-				)
+					(reference "U6")
+					(unit 1)
+				)
+			)
+			(project "NIVARA_ZorionX_BOARD"
+				(path "/8e19332e-3534-4a04-99a8-04957ac8928f/70c9f439-c648-496e-a774-7d3c213f4c72"
+					(reference "U?")
+					(unit 1)
+				)
