File: KiCads del proyecto de Electiva (Nivara_Zorionx)/Salida_Voltaje.kicad_sch (KiCad schematic)
At the start: 5 parts

Commit message: Papadio Dame Fuerza 😭
Parts:
- C11: renamed from C7; footprint (none) -> Capacitor_SMD:C_0805_2012Metric
- C12: renamed from C8; footprint (none) -> Capacitor_SMD:C_0805_2012Metric
- R25: renamed from R23; footprint (none) -> Resistor_SMD:R_0603_1608Metric
- renumbered D3 to D4, U11 to U10
Changed lines of the file:
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@@
 		(on_board yes)
 		(dnp no)
-		(property "Reference" "#PWR049"
+		(property "Reference" "#PWR052"
 			(at 140.97 111.76 0)
 			(effects
@@
 			(project ""
 				(path "/8290cc18-06d0-4e02-a781-29a61ebc321a/9e4d7a0c-a5eb-4e88-9036-0c35e68b279a/11a8222e-f360-40de-9c02-857da7131a56"
-					(reference "#PWR049")
-					(unit 1)
-				)
-			)
-			(project "NIVARA_ZorionX_BOARD"
-				(path "/8e19332e-3534-4a04-99a8-04957ac8928f/11a8222e-f360-40de-9c02-857da7131a56"
-					(reference "#PWR049")
+					(reference "#PWR052")
+					(unit 1)
+				)
+			)
+			(project "NIVARA_ZorionX_BOARD"
+				(path "/8e19332e-3534-4a04-99a8-04957ac8928f/11a8222e-f360-40de-9c02-857da7131a56"
+					(reference "#PWR?")
 					(unit 1)
 				)
@@
 		(dnp no)
 		(fields_autoplaced yes)
-		(property "Reference" "U11"
+		(property "Reference" "U10"
 			(at 143.1133 77.47 0)
 			(effects
@@
 			(project ""
 				(path "/8290cc18-06d0-4e02-a781-29a61ebc321a/9e4d7a0c-a5eb-4e88-9036-0c35e68b279a/11a8222e-f360-40de-9c02-857da7131a56"
-					(reference "U11")
-					(unit 1)
-				)
-			)
-			(project "NIVARA_ZorionX_BOARD"
-				(path "/8e19332e-3534-4a04-99a8-04957ac8928f/11a8222e-f360-40de-9c02-857da7131a56"
-					(reference "U11")
+					(reference "U10")
+					(unit 1)
+				)
+			)
+			(project "NIVARA_ZorionX_BOARD"
+				(path "/8e19332e-3534-4a04-99a8-04957ac8928f/11a8222e-f360-40de-9c02-857da7131a56"
+					(reference "U?")
 					(unit 1)
 				)
@@
 		(dnp no)
 		(fields_autoplaced yes)
-		(property "Reference" "#PWR048"
+		(property "Reference" "#PWR051"
 			(at 140.97 80.01 0)
 			(effects
@@
 			(project ""
 				(path "/8290cc18-06d0-4e02-a781-29a61ebc321a/9e4d7a0c-a5eb-4e88-9036-0c35e68b279a/11a8222e-f360-40de-9c02-857da7131a56"
-					(reference "#PWR048")
-					(unit 1)
-				)
-			)
-			(project "NIVARA_ZorionX_BOARD"
-				(path "/8e19332e-3534-4a04-99a8-04957ac8928f/11a8222e-f360-40de-9c02-857da7131a56"
-					(reference "#PWR048")
+					(reference "#PWR051")
+					(unit 1)
+				)
+			)
+			(project "NIVARA_ZorionX_BOARD"
+				(path "/8e19332e-3534-4a04-99a8-04957ac8928f/11a8222e-f360-40de-9c02-857da7131a56"
+					(reference "#PWR?")
 					(unit 1)
 				)
@@
 		(dnp no)
 		(fields_autoplaced yes)
-		(property "Reference" "#PWR046"
+		(property "Reference" "#PWR054"
 			(at 167.64 66.04 0)
 			(effects
@@
 			(project "NIVARA"
 				(path "/8290cc18-06d0-4e02-a781-29a61ebc321a/9e4d7a0c-a5eb-4e88-9036-0c35e68b279a/11a8222e-f360-40de-9c02-857da7131a56"
-					(reference "#PWR046")
-					(unit 1)
-				)
-			)
-			(project "NIVARA_ZorionX_BOARD"
-				(path "/8e19332e-3534-4a04-99a8-04957ac8928f/11a8222e-f360-40de-9c02-857da7131a56"
-					(reference "#PWR046")
+					(reference "#PWR054")
+					(unit 1)
+				)
+			)
+			(project "NIVARA_ZorionX_BOARD"
+				(path "/8e19332e-3534-4a04-99a8-04957ac8928f/11a8222e-f360-40de-9c02-857da7131a56"
+					(reference "#PWR?")
 					(unit 1)
 				)
@@
 		(dnp no)
 		(fields_autoplaced yes)
-		(property "Reference" "D3"
+		(property "Reference" "D4"
 			(at 170.18 80.0101 90)
 			(effects
@@
 			(project ""
 				(path "/8290cc18-06d0-4e02-a781-29a61ebc321a/9e4d7a0c-a5eb-4e88-9036-0c35e68b279a/11a8222e-f360-40de-9c02-857da7131a56"
-					(reference "D3")
-					(unit 1)
-				)
-			)
-			(project "NIVARA_ZorionX_BOARD"
-				(path "/8e19332e-3534-4a04-99a8-04957ac8928f/11a8222e-f360-40de-9c02-857da7131a56"
-					(reference "D3")
+					(reference "D4")
+					(unit 1)
+				)
+			)
+			(project "NIVARA_ZorionX_BOARD"
+				(path "/8e19332e-3534-4a04-99a8-04957ac8928f/11a8222e-f360-40de-9c02-857da7131a56"
+					(reference "D?")
 					(unit 1)
 				)
@@
 		(on_board yes)
 		(dnp no)
-		(property "Reference" "C7"
+		(property "Reference" "C11"
 			(at 142.24 110.49 90)
 			(effects
@@
 			)
 		)
-		(property "Footprint" ""
+		(property "Footprint" "Capacitor_SMD:C_0805_2012Metric"
 			(at 150.8252 114.3 0)
 			(effects
@@
 			(project ""
 				(path "/8290cc18-06d0-4e02-a781-29a61ebc321a/9e4d7a0c-a5eb-4e88-9036-0c35e68b279a/11a8222e-f360-40de-9c02-857da7131a56"
-					(reference "C7")
-					(unit 1)
-				)
-			)
-			(project "NIVARA_ZorionX_BOARD"
-				(path "/8e19332e-3534-4a04-99a8-04957ac8928f/11a8222e-f360-40de-9c02-857da7131a56"
-					(reference "C7")
+					(reference "C11")
+					(unit 1)
+				)
+			)
+			(project "NIVARA_ZorionX_BOARD"
+				(path "/8e19332e-3534-4a04-99a8-04957ac8928f/11a8222e-f360-40de-9c02-857da7131a56"
+					(reference "C?")
 					(unit 1)
 				)
@@
 		(dnp no)
 		(fields_autoplaced yes)
-		(property "Reference" "#PWR050"
+		(property "Reference" "#PWR053"
 			(at 161.29 100.33 0)
 			(effects
@@
 			(project "NIVARA"
 				(path "/8290cc18-06d0-4e02-a781-29a61ebc321a/9e4d7a0c-a5eb-4e88-9036-0c35e68b279a/11a8222e-f360-40de-9c02-857da7131a56"
-					(reference "#PWR050")
-					(unit 1)
-				)
-			)
-			(project "NIVARA_ZorionX_BOARD"
-				(path "/8e19332e-3534-4a04-99a8-04957ac8928f/11a8222e-f360-40de-9c02-857da7131a56"
-					(reference "#PWR050")
+					(reference "#PWR053")
+					(unit 1)
+				)
+			)
+			(project "NIVARA_ZorionX_BOARD"
+				(path "/8e19332e-3534-4a04-99a8-04957ac8928f/11a8222e-f360-40de-9c02-857da7131a56"
+					(reference "#PWR?")
 					(unit 1)
 				)
@@
 		(on_board yes)
 		(dnp no)
-		(property "Reference" "C8"
+		(property "Reference" "C12"
 			(at 168.91 87.63 90)
 			(effects
@@
 			)
 		)
-		(property "Footprint" ""
+		(property "Footprint" "Capacitor_SMD:C_0805_2012Metric"
 			(at 160.3248 83.82 0)
 			(effects
@@
 			(project "NIVARA"
 				(path "/8290cc18-06d0-4e02-a781-29a61ebc321a/9e4d7a0c-a5eb-4e88-9036-0c35e68b279a/11a8222e-f360-40de-9c02-857da7131a56"
-					(reference "C8")
-					(unit 1)
-				)
-			)
-			(project "NIVARA_ZorionX_BOARD"
-				(path "/8e19332e-3534-4a04-99a8-04957ac8928f/11a8222e-f360-40de-9c02-857da7131a56"
-					(reference "C8")
+					(reference "C12")
+					(unit 1)
+				)
+			)
+			(project "NIVARA_ZorionX_BOARD"
+				(path "/8e19332e-3534-4a04-99a8-04957ac8928f/11a8222e-f360-40de-9c02-857da7131a56"
+					(reference "C?")
 					(unit 1)
 				)
@@
 		(dnp no)
 		(fields_autoplaced yes)
-		(property "Reference" "R23"
+		(property "Reference" "R25"
 			(at 140.97 113.03 90)
 			(effects
@@
 			)
 		)
-		(property "Footprint" ""
+		(property "Footprint" "Resistor_SMD:R_0603_1608Metric"
 			(at 140.97 121.158 90)
 			(effects
@@
 			(project ""
 				(path "/8290cc18-06d0-4e02-a781-29a61ebc321a/9e4d7a0c-a5eb-4e88-9036-0c35e68b279a/11a8222e-f360-40de-9c02-857da7131a56"
-					(reference "R23")
-					(unit 1)
-				)
-			)
-			(project "NIVARA_ZorionX_BOARD"
-				(path "/8e19332e-3534-4a04-99a8-04957ac8928f/11a8222e-f360-40de-9c02-857da7131a56"
-					(reference "R23")
-					(unit 1)
-				)
+					(reference "R25")
+					(unit 1)
+				)
+			)
+			(project "NIVARA_ZorionX_BOARD"
+				(path "/8e19332e-3534-4a04-99a8-04957ac8928f/11a8222e-f360-40de-9c02-857da7131a56"
+					(reference "R?")
+					(unit 1)
+				)
