File: KiCads del proyecto de Electiva (Nivara_Zorionx)/Salidas_PNP.kicad_sch (KiCad schematic)
At the start: 4 parts

Commit message: Papadio Dame Fuerza 😭
Parts:
- R30: renamed from R29; footprint (none) -> Resistor_SMD:R_0603_1608Metric
- R31: renamed from R30; footprint (none) -> Resistor_SMD:R_0603_1608Metric
Changed lines of the file:
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@@
 			(project "NIVARA_ZorionX_BOARD"
 				(path "/8e19332e-3534-4a04-99a8-04957ac8928f/75a26718-4d1a-4f94-8a92-dbb42fb796de"
-					(reference "U14")
+					(reference "U?")
 					(unit 1)
 				)
@@
 			(project "NIVARA_ZorionX_BOARD"
 				(path "/8e19332e-3534-4a04-99a8-04957ac8928f/75a26718-4d1a-4f94-8a92-dbb42fb796de"
-					(reference "U13")
+					(reference "U?")
 					(unit 1)
 				)
@@
 		(dnp no)
 		(fields_autoplaced yes)
-		(property "Reference" "#PWR056"
+		(property "Reference" "#PWR062"
 			(at 133.35 107.95 0)
 			(effects
@@
 			(project "NIVARA"
 				(path "/8290cc18-06d0-4e02-a781-29a61ebc321a/9e4d7a0c-a5eb-4e88-9036-0c35e68b279a/75a26718-4d1a-4f94-8a92-dbb42fb796de"
-					(reference "#PWR056")
-					(unit 1)
-				)
-			)
-			(project "NIVARA_ZorionX_BOARD"
-				(path "/8e19332e-3534-4a04-99a8-04957ac8928f/75a26718-4d1a-4f94-8a92-dbb42fb796de"
-					(reference "#PWR056")
+					(reference "#PWR062")
+					(unit 1)
+				)
+			)
+			(project "NIVARA_ZorionX_BOARD"
+				(path "/8e19332e-3534-4a04-99a8-04957ac8928f/75a26718-4d1a-4f94-8a92-dbb42fb796de"
+					(reference "#PWR?")
 					(unit 1)
 				)
@@
 		(dnp no)
 		(fields_autoplaced yes)
-		(property "Reference" "#PWR057"
+		(property "Reference" "#PWR064"
 			(at 153.67 92.71 0)
 			(effects
@@
 			(project "NIVARA"
 				(path "/8290cc18-06d0-4e02-a781-29a61ebc321a/9e4d7a0c-a5eb-4e88-9036-0c35e68b279a/75a26718-4d1a-4f94-8a92-dbb42fb796de"
-					(reference "#PWR057")
-					(unit 1)
-				)
-			)
-			(project "NIVARA_ZorionX_BOARD"
-				(path "/8e19332e-3534-4a04-99a8-04957ac8928f/75a26718-4d1a-4f94-8a92-dbb42fb796de"
-					(reference "#PWR057")
+					(reference "#PWR064")
+					(unit 1)
+				)
+			)
+			(project "NIVARA_ZorionX_BOARD"
+				(path "/8e19332e-3534-4a04-99a8-04957ac8928f/75a26718-4d1a-4f94-8a92-dbb42fb796de"
+					(reference "#PWR?")
 					(unit 1)
 				)
@@
 		(dnp no)
 		(fields_autoplaced yes)
-		(property "Reference" "#PWR033"
+		(property "Reference" "#PWR061"
 			(at 132.08 83.82 0)
 			(effects
@@
 			(project "NIVARA"
 				(path "/8290cc18-06d0-4e02-a781-29a61ebc321a/9e4d7a0c-a5eb-4e88-9036-0c35e68b279a/75a26718-4d1a-4f94-8a92-dbb42fb796de"
-					(reference "#PWR033")
-					(unit 1)
-				)
-			)
-			(project "NIVARA_ZorionX_BOARD"
-				(path "/8e19332e-3534-4a04-99a8-04957ac8928f/75a26718-4d1a-4f94-8a92-dbb42fb796de"
-					(reference "#PWR033")
+					(reference "#PWR061")
+					(unit 1)
+				)
+			)
+			(project "NIVARA_ZorionX_BOARD"
+				(path "/8e19332e-3534-4a04-99a8-04957ac8928f/75a26718-4d1a-4f94-8a92-dbb42fb796de"
+					(reference "#PWR?")
 					(unit 1)
 				)
@@
 		(dnp no)
 		(fields_autoplaced yes)
-		(property "Reference" "R30"
+		(property "Reference" "R31"
 			(at 125.73 86.36 90)
 			(effects
@@
 			)
 		)
-		(property "Footprint" ""
+		(property "Footprint" "Resistor_SMD:R_0603_1608Metric"
 			(at 125.73 94.488 90)
 			(effects
@@
 			(project "NIVARA"
 				(path "/8290cc18-06d0-4e02-a781-29a61ebc321a/9e4d7a0c-a5eb-4e88-9036-0c35e68b279a/75a26718-4d1a-4f94-8a92-dbb42fb796de"
-					(reference "R30")
-					(unit 1)
-				)
-			)
-			(project "NIVARA_ZorionX_BOARD"
-				(path "/8e19332e-3534-4a04-99a8-04957ac8928f/75a26718-4d1a-4f94-8a92-dbb42fb796de"
-					(reference "R30")
+					(reference "R31")
+					(unit 1)
+				)
+			)
+			(project "NIVARA_ZorionX_BOARD"
+				(path "/8e19332e-3534-4a04-99a8-04957ac8928f/75a26718-4d1a-4f94-8a92-dbb42fb796de"
+					(reference "R?")
 					(unit 1)
 				)
@@
 		(dnp no)
 		(fields_autoplaced yes)
-		(property "Reference" "R29"
+		(property "Reference" "R30"
 			(at 124.46 62.23 90)
 			(effects
@@
 			)
 		)
-		(property "Footprint" ""
+		(property "Footprint" "Resistor_SMD:R_0603_1608Metric"
 			(at 124.46 70.358 90)
 			(effects
@@
 			(project "NIVARA"
 				(path "/8290cc18-06d0-4e02-a781-29a61ebc321a/9e4d7a0c-a5eb-4e88-9036-0c35e68b279a/75a26718-4d1a-4f94-8a92-dbb42fb796de"
-					(reference "R29")
-					(unit 1)
-				)
-			)
-			(project "NIVARA_ZorionX_BOARD"
-				(path "/8e19332e-3534-4a04-99a8-04957ac8928f/75a26718-4d1a-4f94-8a92-dbb42fb796de"
-					(reference "R29")
+					(reference "R30")
+					(unit 1)
+				)
+			)
+			(project "NIVARA_ZorionX_BOARD"
+				(path "/8e19332e-3534-4a04-99a8-04957ac8928f/75a26718-4d1a-4f94-8a92-dbb42fb796de"
+					(reference "R?")
 					(unit 1)
 				)
@@
 		(dnp no)
 		(fields_autoplaced yes)
-		(property "Reference" "#PWR051"
+		(property "Reference" "#PWR063"
 			(at 152.4 68.58 0)
 			(effects
@@
 			(project "NIVARA"
 				(path "/8290cc18-06d0-4e02-a781-29a61ebc321a/9e4d7a0c-a5eb-4e88-9036-0c35e68b279a/75a26718-4d1a-4f94-8a92-dbb42fb796de"
-					(reference "#PWR051")
-					(unit 1)
-				)
-			)
-			(project "NIVARA_ZorionX_BOARD"
-				(path "/8e19332e-3534-4a04-99a8-04957ac8928f/75a26718-4d1a-4f94-8a92-dbb42fb796de"
-					(reference "#PWR051")
-					(unit 1)
-				)
+					(reference "#PWR063")
+					(unit 1)
+				)
+			)
+			(project "NIVARA_ZorionX_BOARD"
+				(path "/8e19332e-3534-4a04-99a8-04957ac8928f/75a26718-4d1a-4f94-8a92-dbb42fb796de"
+					(reference "#PWR?")
+					(unit 1)
+				)
