File: KiCads del proyecto de Electiva (Nivara_Zorionx)/NIVARA_ZorionX.kicad_pcb (KiCad board)
At the start: 2 copper layers, 109.1 x 87.7 mm, 49 parts, among them J1 Screw_Terminal_01x02, J12 Screw_Terminal_01x04, J13 Screw_Terminal_01x02, J14 Screw_Terminal_01x06, J2 Screw_Terminal_01x04, J3 Screw_Terminal_01x02, J4 Screw_Terminal_01x02, J5 Screw_Terminal_01x03, J6 Screw_Terminal_01x02, J9 Screw_Terminal_01x03, K1 G2RL-1, K2 G2RL-1, U1 ESP32-S3-WROOM-1, U10 LTV-357TB, U15 LTV-357TB, U2 AP63200WU, U2 AP63203WU, U4 LTV-357TB, U7 LTV-357TB, U8 LTV-357TB, U9 LTV-357TB

Commit message: Papadio Dame Fuerza 😭
Parts:
- removed the D4 at (166.9, 88.0)
- removed D5: SMF24A, Diode_SMD:D_SMF
- removed J12: Screw_Terminal_01x04, TerminalBlock_Phoenix:TerminalBlock_Phoenix_PT-1,5-4-5.0-H_1x04_P5.00mm_Horizontal
- removed J13: Screw_Terminal_01x02, TerminalBlock_Phoenix:TerminalBlock_Phoenix_PT-1,5-2-5.0-H_1x02_P5.00mm_Horizontal
- removed J14: Screw_Terminal_01x06, TerminalBlock_Phoenix:TerminalBlock_Phoenix_PT-1,5-6-5.0-H_1x06_P5.00mm_Horizontal
- removed the R18 at (176.9, 103.4)
- removed R36: 910, Resistor_SMD:R_0603_1608Metric
- removed the U10 at (170.0, 110.2)
- removed U15: LTV-357TB, Package_SO:SO-4_4.4x3.6mm_P2.54mm
- removed the U2 at (209.0, 89.4)
- removed the U2 at (153.9, 99.1)
- removed the U4 at (185.9, 88.6)
- removed the U4 at (208.8, 103.5)
- removed the U6 at (169.3, 93.6)
- removed the U9 at (170.0, 104.9)
- added C1: 1uF, Capacitor_SMD:C_0805_2012Metric, F.Cu at (121.0, 46.6)
- added C10: 100nF, Capacitor_SMD:C_0805_2012Metric, F.Cu at (111.7, 46.6)
- added C11: 1uF, Capacitor_SMD:C_0805_2012Metric, F.Cu at (123.8, 85.9)
- added C12: 100nF, Capacitor_SMD:C_0805_2012Metric, F.Cu at (106.4, 43.9)
- added C5: 22uF, Capacitor_SMD:C_0805_2012Metric, F.Cu at (77.0, 79.9)
- added C6: 22uF, Capacitor_SMD:C_0805_2012Metric, F.Cu at (77.0, 84.6)
- added C7: 100nF, Capacitor_SMD:C_0805_2012Metric, F.Cu at (54.0, 95.0)
- added C8: 100nF, Capacitor_SMD:C_0805_2012Metric, F.Cu at (57.3, 40.4)
- added C9: 100nF, Capacitor_SMD:C_0805_2012Metric, F.Cu at (64.9, 95.4)
- added J10: Screw_Terminal_01x03, TerminalBlock_Phoenix:TerminalBlock_Phoenix_MKDS-1,5-3_1x03_P5.00mm_Horizontal, F.Cu at (67.1, 32.4)
- added J11: Screw_Terminal_01x03, TerminalBlock_Phoenix:TerminalBlock_Phoenix_MKDS-1,5-3_1x03_P5.00mm_Horizontal, F.Cu at (50.7, 32.3)
- added J7: Screw_Terminal_01x03, TerminalBlock_Phoenix:TerminalBlock_Phoenix_MKDS-1,5-3_1x03_P5.00mm_Horizontal, F.Cu at (124.0, 32.4)
- added J8: Screw_Terminal_01x04, TerminalBlock_Phoenix:TerminalBlock_Phoenix_MKDS-1,5-4_1x04_P5.00mm_Horizontal, F.Cu at (107.2, 32.4)
- added R1: 10k, Resistor_SMD:R_0603_1608Metric, F.Cu at (67.3, 69.3)
- added R10: 910, Resistor_SMD:R_0603_1608Metric, F.Cu at (44.4, 75.8)
- added R11: 412, Resistor_SMD:R_0603_1608Metric, F.Cu at (71.7, 79.2)
- added R12: 412, Resistor_SMD:R_0603_1608Metric, F.Cu at (52.1, 78.8)
- added R13: 120, Resistor_SMD:R_0603_1608Metric, F.Cu at (49.9, 96.1)
- added R14: 120, Resistor_SMD:R_0603_1608Metric, F.Cu at (57.3, 42.9)
- added R15: 100, Resistor_SMD:R_0603_1608Metric, F.Cu at (88.5, 68.6)
- added R16: 100, Resistor_SMD:R_0603_1608Metric, F.Cu at (89.0, 73.2)
- added R20: 412, Resistor_SMD:R_0603_1608Metric, F.Cu at (104.0, 78.0)
- added R21: 160k, Resistor_SMD:R_0603_1608Metric, F.Cu at (78.9, 95.1)
- added R22: 13k, Resistor_SMD:R_0603_1608Metric, F.Cu at (79.0, 89.8)
- added R23: 51k, Resistor_SMD:R_0603_1608Metric, F.Cu at (73.1, 95.3)
- added R24: 16k, Resistor_SMD:R_0603_1608Metric, F.Cu at (73.8, 89.9)
- added R25: 10k, Resistor_SMD:R_0603_1608Metric, F.Cu at (132.4, 84.7)
- added R26: 910, Resistor_SMD:R_0603_1608Metric, F.Cu at (55.3, 75.6)
- added R27: 910, Resistor_SMD:R_0603_1608Metric, F.Cu at (55.3, 84.3)
- added R28: 412, Resistor_SMD:R_0603_1608Metric, F.Cu at (66.8, 74.8)
- added R29: 412, Resistor_SMD:R_0603_1608Metric, F.Cu at (71.6, 83.8)
- added R30: 100, Resistor_SMD:R_0603_1608Metric, F.Cu at (89.0, 77.7)
- added R31: 100, Resistor_SMD:R_0603_1608Metric, F.Cu at (88.9, 82.3)
- added R4: 10k, Resistor_SMD:R_0603_1608Metric, F.Cu at (116.0, 46.6)
- added R5: 196k, Resistor_SMD:R_0603_1608Metric, F.Cu at (81.2, 70.6)
- added R6: 62k, Resistor_SMD:R_0603_1608Metric, F.Cu at (81.2, 76.6)
- added R8: 120, Resistor_SMD:R_0603_1608Metric, F.Cu at (128.5, 38.4)
- added R9: 910, Resistor_SMD:R_0603_1608Metric, F.Cu at (40.9, 100.7)
- added REF**: KiCad-Logo2_5mm_Copper, Symbol:KiCad-Logo2_5mm_Copper, F.Cu at (36.5, 94.1)
- added U11: LTV-357TB, Package_SO:SO-4_4.4x3.6mm_P2.54mm, F.Cu at (62.1, 81.7)
- added U12: LTV-357TB, Package_SO:SO-4_4.4x3.6mm_P2.54mm, F.Cu at (62.1, 89.4)
- added U4: LTV-357TB, Package_SO:SO-4_4.4x3.6mm_P2.54mm, F.Cu at (48.2, 90.5)
- added U5: LTV-357TB, Package_SO:SO-4_4.4x3.6mm_P2.54mm, F.Cu at (48.3, 83.3)
- C2: value 22uf -> 10uF
- C3: value 10mf -> 100nF; footprint Capacitor_SMD:C_1206_3216Metric -> Capacitor_SMD:C_0805_2012Metric
- C4: value 100nf -> 100pF; footprint Capacitor_SMD:C_0603_1608Metric -> Capacitor_SMD:C_0805_2012Metric
- J1, J4: value Screw_Terminal_01x02 -> Screw_Terminal_01x03; footprint TerminalBlock_Phoenix:TerminalBlock_Phoenix_PT-1,5-2-5.0-H_1x02_P5.00mm_Horizontal -> TerminalBlock_Phoenix:TerminalBlock_Phoenix_MKDS-1,5-3_1x03_P5.00mm_Horizontal
- J2: value Screw_Terminal_01x04 -> Screw_Terminal_01x03; footprint TerminalBlock_Phoenix:TerminalBlock_Phoenix_PT-1,5-4-5.0-H_1x04_P5.00mm_Horizontal -> TerminalBlock_Phoenix:TerminalBlock_Phoenix_MKDS-1,5-3_1x03_P5.00mm_Horizontal
- J3: value Screw_Terminal_01x02 -> Screw_Terminal_01x04; footprint TerminalBlock_Phoenix:TerminalBlock_Phoenix_PT-1,5-2-5.0-H_1x02_P5.00mm_Horizontal -> TerminalBlock_Phoenix:TerminalBlock_Phoenix_MKDS-1,5-4_1x04_P5.00mm_Horizontal
- J5: value Screw_Terminal_01x03 -> Screw_Terminal_01x02; footprint TerminalBlock_Phoenix:TerminalBlock_Phoenix_PT-1,5-3-3.5-H_1x03_P3.50mm_Horizontal -> TerminalBlock_Phoenix:TerminalBlock_Phoenix_MKDS-1,5-2_1x02_P5.00mm_Horizontal
- J6: footprint TerminalBlock_Phoenix:TerminalBlock_Phoenix_PT-1,5-2-5.0-H_1x02_P5.00mm_Horizontal -> TerminalBlock_Phoenix:TerminalBlock_Phoenix_MKDS-1,5-2_1x02_P5.00mm_Horizontal
- J9: value Screw_Terminal_01x03 -> Screw_Terminal_01x06; footprint TerminalBlock_Phoenix:TerminalBlock_Phoenix_PT-1,5-3-3.5-H_1x03_P3.50mm_Horizontal -> TerminalBlock_TE-Connectivity:TerminalBlock_TE_282834-6_1x06_P2.54mm_Horizontal
- L1: value L_Iron -> 6.8uH; footprint Inductor_SMD:L_Bourns-SRN6028 -> Inductor_SMD:L_1206_3216Metric
- R19: value 910 -> 412
- R2, R3: value R_US -> 4.7k
- R7: value 910 -> 120
- moved K2 132.8 mm to (38.2, 70.4), turned to 90 degrees
- moved R3 121.9 mm to (40.1, 80.0)
- moved R2 121.7 mm to (40.1, 75.8)
- moved R7 116.8 mm to (79.9, 57.2)
- moved K1 113.5 mm to (38.3, 55.5), turned to 90 degrees
- moved J5 101.9 mm to (109.7, 107.5)
- moved JP1 95.1 mm to (125.5, 47.2)
- moved R19 88.4 mm to (103.1, 57.3), turned to 180 degrees
- moved C4 87.7 mm to (71.9, 63.4)
- moved C2 85.4 mm to (72.0, 69.0)
- moved U3 84.9 mm to (101.0, 48.8), turned to 180 degrees
- moved L1 83.0 mm to (72.3, 59.5), turned to 180 degrees
- moved D3 82.2 mm to (130.0, 44.1)
- moved U9 80.7 mm to (100.1, 82.5)
- moved C3 79.0 mm to (72.0, 74.3)
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- renumbered D7 to D1, D6 to D2, D2 to D3, D3 to D4, R10 to R17, R12 to R18, U11 to U10, U5 to U6, U12 to U7, U7 to U8, U8 to U9
Connections:
- net /NIVARA_BOARD/DRY_INPUT_INTERFACE/DRY_OUT1 renamed GPIO21
- net /NIVARA_BOARD/RS485_INTERFACE/UART_RX renamed GPIO48
- net /NIVARA_BOARD/RS485_INTERFACE/UART_TX renamed GPIO47
- net /NIVARA_BOARD/RS485_INTERFACE/~{TX}/RX renamed /NIVARA_BOARD/Modulo_RS485/~{TX}/RX
- net /NIVARA_BOARD/VOLTAGE_AOUT_INTERFACE/SEL renamed SPII06
- net /NIVARA_BOARD/~{TRANSMIT}/RECEIVE renamed GPIO46
- C2 pad 1: unconnected-(C2-Pad1) -> GND
- C2 pad 2: unconnected-(C2-Pad2) -> VCC
- C3 pad 1: unconnected-(C3-Pad1) -> Net-(U2-BST)
- C3 pad 2: unconnected-(C3-Pad2) -> Net-(U2-SW)
- C4 pad 1: unconnected-(C4-Pad1) -> Net-(D2-A1)
- C4 pad 2: unconnected-(C4-Pad2) -> Net-(U2-FB)
- D2 pad 1: Net-(D6-A1) -> Net-(D2-A1)
- J1 pad 1: /Board_ZorionX/NPN_IN_2 -> /NIVARA_BOARD/NPN_DINPUT_0
- J1 pad 2: /Board_ZorionX/NPN_in_1 -> /NIVARA_BOARD/NPN_DINPUT_1
- J2 pad 1: /Board_ZorionX/A010_IN1 -> /NIVARA_BOARD/PNP_DINPUT_0
- J2 pad 2: /Board_ZorionX/A420_in1 -> /NIVARA_BOARD/PNP_DINPUT_1
- J2 pad 3: /Board_ZorionX/A032_in1 -> PNPIN_GND
- J3 pad 1: VCC -> /NIVARA_BOARD/+10V_AINPUT
- J3 pad 2: GND -> /NIVARA_BOARD/+32V_AINPUT
- J4 pad 1: /Board_ZorionX/D_IN1 -> /NIVARA_BOARD/DRY_DINPUT_0
- J4 pad 2: /Board_ZorionX/D_IN_2 -> /NIVARA_BOARD/DRY_DINPUT_1
- J5 pad 1: /Board_ZorionX/RS485-B -> /NIVARA_BOARD/~{RUN}/STOP
- J5 pad 2: /Board_ZorionX/RS485-A -> GND
- J6 pad 1: /Board_ZorionX/RUN/Stop -> VCC
- J9 pad 1: /Board_ZorionX/AOUT_420_1 -> /NIVARA_BOARD/RL1_OUTPUT_NO
- J9 pad 2: /Board_ZorionX/AOUT_010_1 -> /NIVARA_BOARD/RL1_OUTPUT_NC
- J9 pad 3: GND -> /NIVARA_BOARD/RL1_COM
- JP1 pad 1: Net-(D6-A1) -> Net-(D2-A1)
- L1 pad 1: unconnected-(L1-Pad1) -> Net-(U2-SW)
- L1 pad 2: unconnected-(L1-Pad2) -> Net-(D2-A1)
- R19 pad 1: /NIVARA_BOARD/PNP_DINPUT_1 -> GPIO10
- R19 pad 2: Net-(R19-Pad2) -> +3.3V
- R2 pad 1: unconnected-(R2-Pad1) -> +3.3V
- R2 pad 2: unconnected-(R2-Pad2) -> GPIO16
- R3 pad 1: unconnected-(R3-Pad1) -> +3.3V
- R3 pad 2: unconnected-(R3-Pad2) -> GPIO16
- R7 pad 1: /NIVARA_BOARD/NPN_DINPUT_1 -> Net-(U3-B)
- R7 pad 2: Net-(R7-Pad2) -> /NIVARA_BOARD/RS485_B
- U1 pad 12: /NIVARA_BOARD/PNP_IN_Mod/NPN_Output0 -> GPIO8
- U1 pad 15: /NIVARA_BOARD/RELAY_INTERFACE/RL2_EN -> GPIO3
- U1 pad 17: /NIVARA_BOARD/PNP_IN_Mod/NPN_Output1 -> GPIO9
- U1 pad 18: /NIVARA_BOARD/DRY_INPUT_INTERFACE/DRY_OUT0 -> GPIO10
- U1 pad 26: /NIVARA_BOARD/NPN_OUT_INTERFACE/NPN_EN1 -> GPIO45
- U1 pad 31: /NIVARA_BOARD/NPN_OUT_INTERFACE/NPN_EN0 -> GPIO38
- U1 pad 38: /NIVARA_BOARD/RELAY_INTERFACE/RL1_EN -> GPIO2
- U1 pad 39: /NIVARA_BOARD/mA_AINPUT -> GPIO1
- U1 pad 4: /NIVARA_BOARD/32V_AIN_INTERFACE/32V_ADC -> GPIO4
- U1 pad 5: /NIVARA_BOARD/10V_AIN_INTERFACE/10V_ADC -> GPIO5
- U1 pad 6: /NIVARA_BOARD/PNP_OUT_INTERFACE/PNP_EN0 -> GPIO6
- U1 pad 7: /NIVARA_BOARD/PNP_OUT_INTERFACE/PNP_EN1 -> GPIO7
- U1 pad 8: /NIVARA_BOARD/VOLTAGE_AOUT_INTERFACE/SDA -> GPIO15
- U1 pad 9: /NIVARA_BOARD/VOLTAGE_AOUT_INTERFACE/SCLK -> GPIO16
- U10 pad 1: /NIVARA_BOARD/VOLTAGE_AOUT_INTERFACE/SCLK -> GPIO16
- U8 pad 4: /NIVARA_BOARD/DRY_INPUT_INTERFACE/DRY_OUT0 -> GPIO10
Routing:
- net VCC: track 0.00 -> 216.4 mm, vias 0 -> 4
- net /NIVARA_BOARD/PNP_DOUTPUT_1: track 0.00 -> 134.5 mm, vias 0 -> 2
- net GPIO16: track 0.00 -> 134.2 mm, vias 0 -> 3
- net GPIO1: track 0.00 -> 134.1 mm, vias 0 -> 3
- net /NIVARA_BOARD/PNP_DOUTPUT_0: track 0.00 -> 126.4 mm, vias 0 -> 2
- net Net-(D2-A1): track 0.00 -> 123.4 mm, vias 0 -> 2
- net GND: track 0.00 -> 112.0 mm, vias 0 -> 46
- net /NIVARA_BOARD/NPN_DOUTPUT_0: track 0.00 -> 105.9 mm, vias 0 -> 2
- net GPIO4: track 0.00 -> 103.0 mm, vias 0 -> 3
- net GPIO5: track 0.00 -> 102.5 mm, vias 0 -> 4
- net /NIVARA_BOARD/VOLTAGE_AOUTPUT: track 0.00 -> 93.1 mm, vias 0 -> 2
- net /NIVARA_BOARD/~{RUN}/STOP: track 0.00 -> 82.6 mm, vias 0 -> 2
- net GPIO8: track 0.00 -> 77.3 mm, vias 0 -> 3
- net /NIVARA_BOARD/RS485_B: track 0.00 -> 74.6 mm, vias 0 -> 3
- net GPIO9: track 0.00 -> 72.2 mm, vias 0 -> 3
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- added copper zone on In1.Cu, net +3.3V
- added copper zone on In2.Cu, net GND
Other:
- copper layers 2 -> 4

Commit message: Papadio Dame Fuerza
Parts:
- added REF**: MountingHole_3.2mm_M3_DIN965_Pad_TopOnly, MountingHole:MountingHole_3.2mm_M3_DIN965_Pad_TopOnly, F.Cu at (36.2, 41.4)
- added REF**: MountingHole_3.2mm_M3_DIN965_Pad_TopOnly, MountingHole:MountingHole_3.2mm_M3_DIN965_Pad_TopOnly, F.Cu at (129.7, 98.8)
- moved R3 74.8 mm to (108.9, 50.7)
- moved R23 68.6 mm to (122.5, 47.7), turned to -90 degrees
- moved R2 63.4 mm to (98.7, 51.5)
- moved C8 63.4 mm to (83.3, 98.2)
- moved R14 63.4 mm to (83.3, 100.7)
- moved R24 63.0 mm to (120.8, 48.1), turned to 90 degrees
- moved D4 58.1 mm to (103.0, 43.5)
- moved R31 56.0 mm to (128.5, 42.8)
- moved D2 48.3 mm to (131.9, 42.8), turned to 90 degrees
- moved U10 47.1 mm to (100.1, 49.2), turned to 90 degrees
- moved R7 39.9 mm to (115.4, 39.0)
- moved R29 38.2 mm to (97.1, 55.3)
- moved R28 33.0 mm to (99.7, 77.7)
- moved R12 32.7 mm to (83.3, 69.0)
- moved R30 31.5 mm to (120.0, 72.2)
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Routing:
- net +3.3V: track 20.2 -> 126.8 mm, vias 12 -> 2
- net GPIO16: track 134.2 -> 31.6 mm
- net GPIO5: track 102.5 -> 12.5 mm, vias 4 -> 0
- net /NIVARA_BOARD/+10V_AINPUT: track 13.0 -> 98.4 mm, vias 1 -> 3
- net /NIVARA_BOARD/VOLTAGE_AOUTPUT: track 93.1 -> 19.7 mm, vias 2 -> 0
- net GPIO38: track 30.3 -> 96.7 mm, vias 2 -> 0
- net /NIVARA_BOARD/RS485_B: track 74.6 -> 12.5 mm, vias 3 -> 0
- net GPIO1: track 134.1 -> 78.7 mm, vias 3 -> 2
- net GND: track 112.0 -> 62.7 mm, vias 46 -> 16
- net GPIO7: track 63.1 -> 16.0 mm, vias 3 -> 2
- net Net-(U10-V5V): track 17.0 -> 62.1 mm, vias 0 -> 3
- net /NIVARA_BOARD/Entradas_NPN/NPN_Output0: track 23.7 -> 67.5 mm, vias 0 -> 2
- net Net-(U3-B): track 4.75 -> 47.2 mm, vias 0 -> 2
- net GPIO6: track 57.1 -> 23.7 mm, vias 3 -> 2
- net /NIVARA_BOARD/Entradas_NPN/NPN_Output1: track 5.01 -> 37.3 mm, vias 0 -> 2
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- added copper zone on B.Cu, net GND
- added copper zone on F.Cu, net GND
- removed copper zone on In2.Cu, net GND
Other:
- outline, holes or cut-outs redrawn
- board text added: "Kennedy El Papi"
- board text added: "Pichardo lo más duro del Sistema"
